File: VNA_Project/Downconverters.kicad_sch (KiCad schematic)
At the start: 0 parts

Commit message: finishing up front end
refining Non RF front end
Other:
- note added: "Downconverter will be fabricated on a separate board for testing purposes currently"
Changed lines of the file:
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@@
 	(generator_version "9.0")
 	(paper "A4")
+	(text "Downconverter will be fabricated on a separate board for testing purposes currently\n"
+		(exclude_from_sim no)
+		(at 55.626 16.256 0)
+		(effects
+			(font
+				(size 1.27 1.27)
+			)
+		)
+	)
 )
