File: VNA_Project/VNA_Project.kicad_sch (KiCad schematic)
At the start: 0 parts

Commit message: DAC
DAC
Other:
- removed sheet DAC
Changed lines of the file:
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@@
 			(color 0 0 0 0.0000)
 		)
-		(property "Sheetname" "DAC"
+		(property "Sheetname" "ADC"
 			(at 160.02 65.3284 0)
 			(effects
@@
 			)
 		)
-		(property "Sheetfile" "DAC.kicad_sch"
+		(property "Sheetfile" "ADC.kicad_sch"
 			(at 160.02 93.2946 0)
-			(effects
-				(font
-					(size 1.27 1.27)
-				)
-				(justify left top)
-			)
-		)
-		(instances
-			(project "VNA_Project"
-				(path "/8b9c6944-c5f7-4a92-a452-dc4fa5f3924d"
-					(page "7")
-				)
-			)
-		)
-	)
-	(sheet
-		(at 189.23 66.04)
-		(size 26.67 26.67)
-		(exclude_from_sim no)
-		(in_bom yes)
-		(on_board yes)
-		(dnp no)
-		(fields_autoplaced yes)
-		(stroke
-			(width 0.1524)
-			(type solid)
-		)
-		(fill
-			(color 0 0 0 0.0000)
-		)
-		(property "Sheetname" "ADC"
-			(at 189.23 65.3284 0)
-			(effects
-				(font
-					(size 1.27 1.27)
-				)
-				(justify left bottom)
-			)
-		)
-		(property "Sheetfile" "ADC.kicad_sch"
-			(at 189.23 93.2946 0)
 			(effects
 				(font
@@
 	)
 	(sheet
-		(at 107.95 104.14)
+		(at 105.41 104.14)
 		(size 25.4 25.4)
 		(exclude_from_sim no)
@@
 		)
 		(property "Sheetname" "Downconverters"
-			(at 107.95 103.4284 0)
+			(at 105.41 103.4284 0)
 			(effects
 				(font
@@
 		)
 		(property "Sheetfile" "Downconverters.kicad_sch"
-			(at 107.95 130.1246 0)
+			(at 105.41 130.1246 0)
 			(effects
 				(font

Commit message: finishing up front end
refining Non RF front end
Other:
- removed sheet Filters
Changed lines of the file:
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@@
-	)
-	(sheet
-		(at 181.61 104.14)
-		(size 25.4 25.4)
-		(exclude_from_sim no)
-		(in_bom yes)
-		(on_board yes)
-		(dnp no)
-		(fields_autoplaced yes)
-		(stroke
-			(width 0.1524)
-			(type solid)
-		)
-		(fill
-			(color 0 0 0 0.0000)
-		)
-		(property "Sheetname" "Filters"
-			(at 181.61 103.4284 0)
-			(effects
-				(font
-					(size 1.27 1.27)
-				)
-				(justify left bottom)
-			)
-		)
-		(property "Sheetfile" "Filters.kicad_sch"
-			(at 181.61 130.1246 0)
-			(effects
-				(font
-					(size 1.27 1.27)
-				)
-				(justify left top)
-			)
-		)
-		(instances
-			(project "VNA_Project"
-				(path "/8b9c6944-c5f7-4a92-a452-dc4fa5f3924d"
-					(page "9")
-				)
-			)
-		)
 	)
 	(sheet
@@
 	)
 	(sheet
-		(at 76.2 104.14)
+		(at 80.01 104.14)
 		(size 25.4 25.4)
 		(exclude_from_sim no)
@@
 		)
 		(property "Sheetname" "VCO"
-			(at 76.2 103.4284 0)
+			(at 80.01 103.4284 0)
 			(effects
 				(font
@@
 		)
 		(property "Sheetfile" "VCO.kicad_sch"
-			(at 76.2 130.1246 0)
+			(at 80.01 130.1246 0)
 			(effects
 				(font
@@
 	)
 	(sheet
-		(at 105.41 104.14)
+		(at 111.76 104.14)
 		(size 25.4 25.4)
 		(exclude_from_sim no)
@@
 		)
 		(property "Sheetname" "Downconverters"
-			(at 105.41 103.4284 0)
+			(at 111.76 103.4284 0)
 			(effects
 				(font
@@
 		)
 		(property "Sheetfile" "Downconverters.kicad_sch"
-			(at 105.41 130.1246 0)
+			(at 111.76 130.1246 0)
 			(effects
 				(font
