File: VNA_Project/VNA_Project.kicad_sch (KiCad schematic)
At the start: 0 parts

Commit message: footprints + initial layout shape
footprints + initial layout shape
Changed lines of the file:
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@@
 	)
 	(sheet
-		(at 129.54 66.04)
+		(at 165.1 65.532)
 		(size 26.67 26.67)
 		(exclude_from_sim no)
@@
 		)
 		(property "Sheetname" "Ethernet"
-			(at 129.54 65.3284 0)
+			(at 165.1 64.8204 0)
 			(effects
 				(font
@@
 		)
 		(property "Sheetfile" "Ethernet.kicad_sch"
-			(at 129.54 93.2946 0)
-			(effects
-				(font
-					(size 1.27 1.27)
-				)
-				(justify left top)
-			)
-		)
-		(instances
-			(project "VNA_Project"
-				(path "/8b9c6944-c5f7-4a92-a452-dc4fa5f3924d"
-					(page "10")
+			(at 165.1 92.7866 0)
+			(effects
+				(font
+					(size 1.27 1.27)
+				)
+				(justify left top)
+			)
+		)
+		(instances
+			(project "VNA_Project"
+				(path "/8b9c6944-c5f7-4a92-a452-dc4fa5f3924d"
+					(page "5")
 				)
 			)
@@
 			(project "VNA_Project"
 				(path "/8b9c6944-c5f7-4a92-a452-dc4fa5f3924d"
-					(page "5")
-				)
-			)
-		)
-	)
-	(sheet
-		(at 99.06 66.04)
+					(page "8")
+				)
+			)
+		)
+	)
+	(sheet
+		(at 99.822 65.532)
 		(size 25.4 26.67)
 		(exclude_from_sim no)
@@
 		)
 		(property "Sheetname" "MCU"
-			(at 99.06 65.3284 0)
+			(at 99.822 64.8204 0)
 			(effects
 				(font
@@
 		)
 		(property "Sheetfile" "MCU_vna.kicad_sch"
-			(at 99.06 93.2946 0)
+			(at 99.822 92.7866 0)
+			(effects
+				(font
+					(size 1.27 1.27)
+				)
+				(justify left top)
+			)
+		)
+		(instances
+			(project "VNA_Project"
+				(path "/8b9c6944-c5f7-4a92-a452-dc4fa5f3924d"
+					(page "3")
+				)
+			)
+		)
+	)
+	(sheet
+		(at 131.572 65.532)
+		(size 25.654 26.67)
+		(exclude_from_sim no)
+		(in_bom yes)
+		(on_board yes)
+		(dnp no)
+		(fields_autoplaced yes)
+		(stroke
+			(width 0.1524)
+			(type solid)
+		)
+		(fill
+			(color 0 0 0 0.0000)
+		)
+		(property "Sheetname" "ADC"
+			(at 131.572 64.8204 0)
+			(effects
+				(font
+					(size 1.27 1.27)
+				)
+				(justify left bottom)
+			)
+		)
+		(property "Sheetfile" "ADC.kicad_sch"
+			(at 131.572 92.7866 0)
 			(effects
 				(font
@@
 				(path "/8b9c6944-c5f7-4a92-a452-dc4fa5f3924d"
 					(page "4")
-				)
-			)
-		)
-	)
-	(sheet
-		(at 160.02 66.04)
-		(size 26.67 26.67)
-		(exclude_from_sim no)
-		(in_bom yes)
-		(on_board yes)
-		(dnp no)
-		(fields_autoplaced yes)
-		(stroke
-			(width 0.1524)
-			(type solid)
-		)
-		(fill
-			(color 0 0 0 0.0000)
-		)
-		(property "Sheetname" "ADC"
-			(at 160.02 65.3284 0)
-			(effects
-				(font
-					(size 1.27 1.27)
-				)
-				(justify left bottom)
-			)
-		)
-		(property "Sheetfile" "ADC.kicad_sch"
-			(at 160.02 93.2946 0)
-			(effects
-				(font
-					(size 1.27 1.27)
-				)
-				(justify left top)
-			)
-		)
-		(instances
-			(project "VNA_Project"
-				(path "/8b9c6944-c5f7-4a92-a452-dc4fa5f3924d"
-					(page "6")
 				)
 			)
@@
 			(project "VNA_Project"
 				(path "/8b9c6944-c5f7-4a92-a452-dc4fa5f3924d"
-					(page "3")
+					(page "6")
 				)
 			)
@@
 			(project "VNA_Project"
 				(path "/8b9c6944-c5f7-4a92-a452-dc4fa5f3924d"
-					(page "8")
-				)
-			)
+					(page "7")
+				)
+			)

Commit message: GRB BOM
GRB BOM
Other:
- sheet ADC renamed ADC [4]
- sheet Directional Coupler renamed Directional Coupler [8]
- sheet Downconverters renamed Downconverters [7]
- sheet Ethernet renamed Ethernet [5]
- sheet MCU renamed MCU [3]
- sheet Power renamed Power [2]
- sheet VCO renamed VCO [6]
Changed lines of the file:
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@@
 			(color 0 0 0 0.0000)
 		)
-		(property "Sheetname" "Power"
+		(property "Sheetname" "Power [2]"
 			(at 68.58 65.3284 0)
 			(effects
 				(font
 					(size 1.27 1.27)
+					(thickness 0.254)
+					(bold yes)
+					(italic yes)
 				)
 				(justify left bottom)
@@
 	)
 	(sheet
-		(at 165.1 65.532)
+		(at 164.846 65.532)
 		(size 26.67 26.67)
 		(exclude_from_sim no)
@@
 			(color 0 0 0 0.0000)
 		)
-		(property "Sheetname" "Ethernet"
-			(at 165.1 64.8204 0)
-			(effects
-				(font
-					(size 1.27 1.27)
+		(property "Sheetname" "Ethernet [5]"
+			(at 164.846 64.8204 0)
+			(effects
+				(font
+					(size 1.27 1.27)
+					(thickness 0.254)
+					(bold yes)
+					(italic yes)
 				)
 				(justify left bottom)
@@
 		)
 		(property "Sheetfile" "Ethernet.kicad_sch"
-			(at 165.1 92.7866 0)
+			(at 164.846 92.7866 0)
 			(effects
 				(font
@@
 			(color 0 0 0 0.0000)
 		)
-		(property "Sheetname" "Directional Coupler"
+		(property "Sheetname" "Directional Coupler [8]"
 			(at 144.78 103.4284 0)
 			(effects
 				(font
 					(size 1.27 1.27)
+					(thickness 0.254)
+					(bold yes)
+					(italic yes)
 				)
 				(justify left bottom)
@@
 			(color 0 0 0 0.0000)
 		)
-		(property "Sheetname" "MCU"
+		(property "Sheetname" "MCU [3]"
 			(at 99.822 64.8204 0)
 			(effects
 				(font
 					(size 1.27 1.27)
+					(thickness 0.254)
+					(bold yes)
+					(italic yes)
 				)
 				(justify left bottom)
@@
 			(color 0 0 0 0.0000)
 		)
-		(property "Sheetname" "ADC"
+		(property "Sheetname" "ADC [4]"
 			(at 131.572 64.8204 0)
 			(effects
 				(font
 					(size 1.27 1.27)
+					(thickness 0.254)
+					(bold yes)
+					(italic yes)
 				)
 				(justify left bottom)
@@
 			(color 0 0 0 0.0000)
 		)
-		(property "Sheetname" "VCO"
+		(property "Sheetname" "VCO [6]"
 			(at 80.01 103.4284 0)
 			(effects
 				(font
 					(size 1.27 1.27)
+					(thickness 0.254)
+					(bold yes)
+					(italic yes)
 				)
 				(justify left bottom)
@@
 			(color 0 0 0 0.0000)
 		)
-		(property "Sheetname" "Downconverters"
+		(property "Sheetname" "Downconverters [7]"
 			(at 111.76 103.4284 0)
 			(effects
 				(font
 					(size 1.27 1.27)
-				)
-				(justify left bottom)
+					(thickness 0.254)
+					(bold yes)
+					(italic yes)
+				)
+				(justify left bottom)
