File: VNA_Project/ADC.kicad_sch (KiCad schematic)
At the start: 0 parts

Commit message: ADC initial
ADC initial
Parts:
- added U3: AD9238BSTZ-20, ST_64_1_ADI, symbol Non_KiCad_Symbols:AD9238BSTZ-20
Changed lines of the file:
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@@
 	(generator "eeschema")
 	(generator_version "9.0")
-	(paper "A4")
+	(paper "A3")
+	(symbol
+		(lib_id "Non_KiCad_Symbols:AD9238BSTZ-20")
+		(at 173.99 88.9 0)
+		(unit 1)
+		(exclude_from_sim no)
+		(in_bom yes)
+		(on_board yes)
+		(dnp no)
+		(fields_autoplaced yes)
+		(property "Reference" "U3"
+			(at 201.93 78.74 0)
+			(effects
+				(font
+					(size 1.524 1.524)
+				)
+			)
+		)
+		(property "Value" "AD9238BSTZ-20"
+			(at 201.93 81.28 0)
+			(effects
+				(font
+					(size 1.524 1.524)
+				)
+			)
+		)
+		(property "Footprint" "ST_64_1_ADI"
+			(at 173.99 88.9 0)
+			(effects
+				(font
+					(size 1.27 1.27)
+					(italic yes)
+				)
+				(hide yes)
+			)
+		)
+		(property "Datasheet" "https://www.analog.com/media/en/technical-documentation/data-sheets/AD9238.pdf"
+			(at 173.99 88.9 0)
+			(effects
+				(font
+					(size 1.27 1.27)
+					(italic yes)
+				)
+				(hide yes)
+			)
+		)
+		(property "Description" ""
+			(at 173.99 88.9 0)
+			(effects
+				(font
+					(size 1.27 1.27)
+				)
+				(hide yes)
+			)
+		)
+		(pin "8"
+		)
+		(pin "1"
+		)
+		(pin "13"
+		)
+		(pin "2"
+		)
+		(pin "3"
+		)
+		(pin "4"
+		)
+		(pin "5"
+		)
+		(pin "6"
+		)
+		(pin "7"
+		)
+		(pin "9"
+		)
+		(pin "10"
+		)
+		(pin "11"
+		)
+		(pin "12"
+		)
+		(pin "27"
+		)
+		(pin "29"
+		)
+		(pin "31"
+		)
+		(pin "18"
+		)
+		(pin "23"
+		)
+		(pin "61"
+		)
+		(pin "59"
+		)
+		(pin "57"
+		)
+		(pin "55"
+		)
+		(pin "54"
+		)
+		(pin "26"
+		)
+		(pin "17"
+		)
+		(pin "19"
+		)
+		(pin "21"
+		)
+		(pin "24"
+		)
+		(pin "14"
+		)
+		(pin "15"
+		)
+		(pin "16"
+		)
+		(pin "20"
+		)
+		(pin "22"
+		)
+		(pin "25"
+		)
+		(pin "28"
+		)
+		(pin "30"
+		)
+		(pin "32"
+		)
+		(pin "64"
+		)
+		(pin "63"
+		)
+		(pin "62"
+		)
+		(pin "60"
+		)
+		(pin "58"
+		)
+		(pin "56"
+		)
+		(pin "48"
+		)
+		(pin "36"
+		)
+		(pin "35"
+		)
+		(pin "34"
+		)
+		(pin "51"
+		)
+		(pin "53"
+		)
+		(pin "45"
+		)
+		(pin "42"
+		)
+		(pin "33"
+		)
+		(pin "37"
+		)
+		(pin "52"
+		)
+		(pin "39"
+		)
+		(pin "40"
+		)
+		(pin "43"
+		)
+		(pin "47"
+		)
+		(pin "49"
+		)
+		(pin "41"
+		)
+		(pin "44"
+		)
+		(pin "46"
+		)
+		(pin "38"
+		)
+		(pin "50"
+		)
+		(instances
+			(project ""
+				(path "/8b9c6944-c5f7-4a92-a452-dc4fa5f3924d/e352f3b5-433e-42a1-adc5-ff1237016ad8"
+					(reference "U3")
+					(unit 1)
+				)
+			)
+		)
+	)
 )

Commit message: ADC AA filter
ADC AA Filter
Parts:
- added C12, C14, C15, C17, C19, C21, C23, C24: 100p, symbol Device:C_Small
- added C13, C16, C20, C22: 15p, symbol Device:C_Small
- added R17, R20, R23, R28: 18, symbol Device:R_Small
- added R18, R21, R24, R27: 51, symbol Device:R_Small
- added R19, R22, R25, R26: 30, symbol Device:R_Small
- added U4, U5: LT1813CS8-TRPBF, SO-8_S_LIT, symbol Non_KiCad_Symbols:LT1813CS8-TRPBF
Connections:
- new net: C17.1, R21.2, R22.1
- new net: C21.1, R24.2, R25.1
- new net: C20.1, R25.2, U5.3 (+INA)
- new net: C22.1, R26.2, U5.5 (+INB)
- new net: C12.1, R17.2, R18.1
- new net: C15.1, R20.2, R21.1
- new net: C16.1, R22.2, U4.5 (+INB)
- new net: C14.1, R18.2, R19.1
- new net: C24.1, R27.1, R28.2
- new net: C23.1, R26.1, R27.2
- new net: C13.1, R19.2, U4.3 (+INA)
- new net: C19.1, R23.2, R24.1
- new net GND: C12.2, C13.2, C15.2, C16.2, C19.2, C20.2, C22.2, C24.2
- new net OP_AMP_BIAS-: U4.4 (V-), U5.4 (V-)
- new net OUTA: C14.2, R20.1, U4.1 (OUTA), U4.2 (-INA)
- new net OUTA2: C21.2, R28.1, U5.1 (OUTA), U5.2 (-INA)
- new net OUTB: C17.2, U4.6 (-INB), U4.7 (OUTB)
- new net OUTB2: C23.2, U5.6 (-INB), U5.7 (OUTB)
- new net VNA_A_WAVE: R17.1
- new net VNA_B_WAVE: R23.1
Other:
- note added: "AA Filter Ideal Simulation, GBP is 100 MHz and slew rate is sufficient, might be a bit lazy to import the actual op amp into LTSPICE, might revisit"
- note added: "Cascaded Sallen Key Anti-Aliasing Filter, fc = 10MHz, 20MSPS"
- note added: "One dual ADC per directional coupler"
- note added: "S11"
- note added: "VNA_A_WAVE"
- note added: "VNA_B_WAVE"
- moved on the sheet: U3

Commit message: minor changes
minor changes
Connections:
- no-connect marks 0 -> 3
Other:
- moved on the sheet: U3
Changed lines of the file:
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@@
 	)
 	(junction
+		(at 118.11 35.56)
+		(diameter 0)
+		(color 0 0 0 0)
+	)
+	(junction
 		(at 161.29 38.1)
 		(diameter 0)
@@
 		(color 0 0 0 0)
 	)
+	(no_connect
+		(at 156.21 201.93)
+	)
+	(no_connect
+		(at 156.21 204.47)
+	)
+	(no_connect
+		(at 100.33 207.01)
+	)
 	(wire
 		(pts
@@
 	(wire
 		(pts
+			(xy 118.11 31.75) (xy 118.11 35.56)
+		)
+		(stroke
+			(width 0)
+			(type default)
+		)
+	)
+	(wire
+		(pts
 			(xy 90.17 88.9) (xy 90.17 90.17)
 		)
@@
 	(global_label "OUTA"
 		(shape input)
-		(at 118.11 35.56 90)
+		(at 118.11 31.75 90)
 		(fields_autoplaced yes)
 		(effects
@@
 		)
 		(property "Intersheetrefs" "${INTERSHEET_REFS}"
-			(at 118.11 27.8576 90)
+			(at 118.11 24.0476 90)
 			(effects
 				(font
@@
 	(symbol
 		(lib_id "Non_KiCad_Symbols:AD9238BSTZ-20")
-		(at 50.8 151.13 0)
+		(at 100.33 148.59 0)
 		(unit 1)
 		(exclude_from_sim no)
@@
 		(fields_autoplaced yes)
 		(property "Reference" "U3"
-			(at 78.74 140.97 0)
+			(at 171.45 143.256 0)
 			(effects
 				(font
@@
 		)
 		(property "Value" "AD9238BSTZ-20"
-			(at 78.74 143.51 0)
+			(at 159.004 143.002 0)
 			(effects
 				(font
@@
 		)
 		(property "Footprint" "ST_64_1_ADI"
-			(at 50.8 151.13 0)
+			(at 127.254 149.606 0)
 			(effects
 				(font
@@
 		)
 		(property "Datasheet" "https://www.analog.com/media/en/technical-documentation/data-sheets/AD9238.pdf"
-			(at 50.8 151.13 0)
+			(at 127.762 157.988 0)
 			(effects
 				(font
@@
 		)
 		(property "Description" ""
-			(at 50.8 151.13 0)
+			(at 100.33 148.59 0)
 			(effects
 				(font

Commit message: adc
adc
Parts:
- added C601, C602, C603: 0.1u, symbol Device:C
- added C604, C605, C606: 10u, symbol Device:C
Connections:
- net GND: now also C601.2, C602.2, C603.2, C604.2, C605.2, C606.2
- net +3.3V: now reaches U3.29 (DRVDD)
- net +3.3V: now also U3.41 (DRVDD), U3.52 (DRVDD), C601.1, C602.1, C603.1, C604.1, C605.1, C606.1
- no-connect marks 3 -> 4
Other:
- moved on the sheet: U3

Commit message: adc
adc
Parts:
- added C27, C28, C29, C31: 0.1u, symbol Device:C
- added C30: 10u, symbol Device:C
- added C32, C33: 100p, symbol Device:C_Small
- added FB1, FB2: FerriteBead, symbol Device:FerriteBead
- added R30, R31, R32, R33, R34, R35, R36, R37: 499, symbol Device:R_Small
- added U7, U8: AD8138ARZ, R_8_ADI, symbol Non_KiCad_Symbols:AD8138ARZ
Connections:
- net GND: now also U3.1 (AGND), U3.13 (AGND), U3.16 (AGND), U3.28 (DRGND), U3.4 (AGND), U3.40 (DRGND), U3.53 (DRGND), C27.2, C28.2, C29.2, C30.2, C31.2, C32.2, C33.2, R31.1, R34.1, U7.6 (V-), U8.6 (V-)
- net OUTA: now also R30.1
- net OUTA2: now also R37.1
- net at U3.12 (AVDD): now also U3.17 (AVDD), U3.5 (AVDD), U3.64 (AVDD), C27.1, C28.1, C29.1, C31.1, FB2.2
- net diffout2_-: now reaches U3.14 (VIN-_B)
- net diffout2_-: now also R36.2, U8.5 (-OUT)
- net diffout2_+: now reaches U3.15 (VIN+_B)
- net diffout2_+: now also R35.2, U8.4 (+OUT)
- net diffout_+: now reaches U3.2 (VIN+_A)
- net diffout_+: now also R32.2, U7.4 (+OUT)
- net D0_B: now reaches U3.25 (D0_B)
- net D1_B: now reaches U3.26 (D1_B)
- net D2_B: now reaches U3.27 (D2_B)
- net diffout_-: now reaches U3.3 (VIN-_A)
- net diffout_-: now also R33.2, U7.5 (-OUT)
- net D3_B: now reaches U3.30 (D3_B)
- net D4_B: now reaches U3.31 (D4_B)
- net D5_B: now reaches U3.32 (D5_B)
- net D6_B: now reaches U3.33 (D6_B)
- net D7_B: now reaches U3.34 (D7_B)
- net D8_B: now reaches U3.35 (D8_B)
- net D9_B: now reaches U3.36 (D9_B)
- net D10_B: now reaches U3.37 (D10_B)
- net D11_B: now reaches U3.38 (D11_B)
- net D0_A: now reaches U3.44 (D0_A)
- net D1_A: now reaches U3.45 (D1_A)
- net D2_A: now reaches U3.46 (D2_A)
- net D3_A: now reaches U3.47 (D3_A)
- net D4_A: now reaches U3.48 (D4_A)
- net D5_A: now reaches U3.49 (D5_A)
- net D6_A: now reaches U3.50 (D6_A)
- net D7_A: now reaches U3.51 (D7_A)
- net D8_A: now reaches U3.54 (D8_A)
- net D9_A: now reaches U3.55 (D9_A)
- net D10_A: now reaches U3.56 (D10_A)
- net D11_A: now reaches U3.57 (D11_A)
- net +3.3V: no longer names the net of C601.1, C602.1, C603.1, C604.1, C605.1, C606.1, U3.29 (DRVDD), U3.41 (DRVDD), U3.52 (DRVDD)
- net +3.3V: now also FB1.1
- new net: R36.1, R37.2, U8.8 (+IN)
- new net: R34.2, R35.1, U8.1 (-IN)
- new net: R31.2, R32.1, U7.1 (-IN)
- new net: R30.2, R33.1, U7.8 (+IN)
- new net +3V0: C30.1, FB1.2, FB2.1
- new net VCC: U7.3 (V+), U8.3 (V+)
- new net VREF_ADCD: C32.1, C33.1, U7.2 (VOCM), U8.2 (VOCM)
- no-connect marks 4 -> 6
Other:
- note added: "typical power dissipation of 12 mW"
- moved on the sheet: C601, C602, C603, C604, C605, C606, U3

Commit message: finishing up front end
refining Non RF front end
Parts:
- added C18, C40, C42, C43: 0.1u, symbol Device:C
- added C41, C44: 10u, symbol Device:C
- added J2, J4, J6: Conn_Coaxial, symbol Connector:Conn_Coaxial
- added R5: 50, symbol Device:R
- added SW2, SW4, SW5: SW_SPDT, symbol Switch:SW_SPDT
Connections:
- net OP_AMP_BIAS- is gone; now on net GND: U4.4 (V-), U5.4 (V-)
- net VCC is gone; now on net +5V: U7.3 (V+), U8.3 (V+)
- net +3V0: now also U3.62 (SHARED_REF), SW2.1 (A), SW4.1 (A), SW5.1 (A)
- net GND: now also U3.19 (DCS), U3.21 (PDWN_B), U3.60 (PDWN_A), U3.9 (SENSE), C18.2, C42.2, C43.2, C44.2, J2.2 (Ext), J4.1 (In), J6.1 (In), R5.2, SW2.3 (C), SW4.3 (C), SW5.3 (C)
- net +5V: now reaches U5.8 (V+)
- net +5V: now also U4.8 (V+)
- net at U3.10 (REFB_B): now also U3.7 (REFB_A), C40.2, C41.2, C42.1
- net at U3.11 (REFT_B): now also U3.6 (REFT_A), C18.1, C40.1, C41.1
- net clk_a_adc: now reaches U3.18 (CLK_B)
- net clk_a_adc: now also U3.61 (MUX_SELECT), U3.63 (CLK_A), J2.1 (In), R5.1
- net at U3.20 (DFS): now also SW2.2 (B)
- net at U3.22 (OEB_B): now also SW5.2 (B)
- net OTR_B: now reaches U3.39 (OTR_B)
- net OTR_A: now reaches U3.58 (OTR_A)
- net at U3.59 (OEB_A): now also SW4.2 (B)
- net at U3.8 (VREF): now also C43.1, C44.1
- net VNA_A_WAVE: no longer names the net of R17.1
- net VNA_A_WAVE: now also J4.2 (Ext)
- net VNA_B_WAVE: no longer names the net of R23.1
- net VNA_B_WAVE: now also J6.2 (Ext)
Other:
- note added: "+3 for 2s complement, GND for offset binary"
- note added: "Downconverter Output"
- note added: "In all reference configurations, REFT and REFB drive the ADC core and establish its input span. The input range of the ADC always equals twice the voltage at the reference pin for either an internal or an external reference."
- note added: "connect to function generator 20MHz for testing, build own oscillator reference afterwards"
- note removed: "AA Filter Ideal Simulation, GBP is 100 MHz and slew rate is sufficient, might be a bit lazy to import the actual op amp into LTSPICE, might revisit"

Commit message: AA filtering
redoing AA filtering
Parts:
- removed C12, C14, C15, C17, C19, C21, C23, C24: 100p, symbol Device:C_Small
- removed C13, C16, C20, C22: 15p, symbol Device:C_Small
- removed R17, R20, R23, R28: 18, symbol Device:R_Small
- removed R18, R21, R24, R27: 51, symbol Device:R_Small
- removed R19, R22, R25, R26: 30, symbol Device:R_Small
- added C46, C47, C49, C50: 100n, symbol Device:C_Small
- added R8, R9: 50, symbol Device:R_Small
- added TP1, TP2, TP3: TestPoint, symbol Connector:TestPoint
Connections:
- net +5V: now also C46.2, C47.2, C49.1, C50.1
- net GND: now also C46.1, C47.1, C49.2, C50.2, R8.1, R9.1
- net OUTA: no longer U4.1 (OUTA), U4.2 (-INA)
- net OUTA2: no longer U5.1 (OUTA), U5.2 (-INA)
- net at C601.1, C602.1, C603.1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: now also TP3.1
- net at C43.1, C44.1, U3.8 (VREF): now also TP1.1
- net at J4.2 (Ext): now also R8.2
- net at C27.1, C28.1, C29.1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: now also TP2.1
- net at J6.2 (Ext): now also R9.2
- net OUTB: no longer names the net of U4.6 (-INB)
- net OUTB: no longer U4.7 (OUTB)
- net OUTB2: no longer names the net of U5.6 (-INB)
- net OUTB2: no longer U5.7 (OUTB)
Other:
- note added: "Cascaded third order Sallen Key Anti-Aliasing Filter, fc = 10MHz, 20MSPS"
- note added: "differential transformers"
- note removed: "Cascaded Sallen Key Anti-Aliasing Filter, fc = 10MHz, 20MSPS"

Commit message: VNA V1
FRONT END  FIRST PROTOTYPE SCHEMATIC DONE
Parts:
- removed J6: Conn_Coaxial, symbol Connector:Conn_Coaxial
- removed R9: 50, symbol Device:R_Small
- added C51, C52: 100n, symbol Device:C_Small
- added C58, C60, C62, C63: 100p, symbol Device:C_Small
- added C59, C61: 12p, symbol Device:C_Small
- added J8: Conn_Coaxial, symbol Connector:Conn_Coaxial
- added R25, R59: 220, symbol Device:R
- added R26, R58: 910, symbol Device:R
- added R27, R57: 300, symbol Device:R
- added R28: 50, symbol Device:R_Small
Connections:
- net +5V: now also C51.2; no longer C46.2
- net GND: now also C51.1, C52.1, C58.1, C59.1, C61.1, C63.1, J8.1 (In), R28.1; no longer U4.4 (V-), U5.4 (V-)
- net OUTA: now also U4.1 (OUTA), U4.2 (-INA), R25.2; no longer R30.1
- net OUTA2: now also U5.1 (OUTA), U5.2 (-INA), R59.2; no longer R37.1
- net at U5.3 (+INA): now also J8.2 (Ext), R28.2
- net at U5.5 (+INB): now also C61.2, R57.1
- net OUTB2: now reaches U5.6 (-INB)
- net OUTB2: now also R37.1, U5.7 (OUTB), C62.1
- net at J4.2 (Ext), R8.2: now also U4.3 (+INA)
- net at U4.5 (+INB): now also C59.2, R27.1
- net OUTB: now reaches U4.6 (-INB)
- net OUTB: now also R30.1, U4.7 (OUTB), C60.1
- new net: C63.2, R58.2, R59.1
- new net: C62.2, R57.2, R58.1
- new net: C60.2, R26.1, R27.2
- new net: C58.2, R25.1, R26.2
- new net -5V: C46.2, C52.2, U4.4 (V-), U5.4 (V-)
Other:
- note added: "8MHz fc sallen key third order AA filter"
- note removed: "Cascaded third order Sallen Key Anti-Aliasing Filter, fc = 10MHz, 20MSPS"
- moved on the sheet: J4, R8
