File: VNA_Project/ADC.kicad_sch (KiCad schematic)
At the start: 64 parts, among them J2 Conn_Coaxial, J4 Conn_Coaxial, J8 Conn_Coaxial, SW2 SW_SPDT, SW4 SW_SPDT, SW5 SW_SPDT, U3 AD9238BSTZ-20, U4 LT1813CS8-TRPBF, U5 LT1813CS8-TRPBF, U7 AD8138ARZ, U8 AD8138ARZ

Commit message: footprints + initial layout shape
footprints + initial layout shape
Parts:
- C401: renamed from C30; footprint (none) -> Capacitor_SMD:C_0603_1608Metric_Pad1.08x0.95mm_HandSolder
- C402: renamed from C31; footprint (none) -> Capacitor_SMD:C_0603_1608Metric_Pad1.08x0.95mm_HandSolder
- C403: renamed from C52; footprint (none) -> Capacitor_SMD:C_0603_1608Metric_Pad1.08x0.95mm_HandSolder
- C404: renamed from C46; footprint (none) -> Capacitor_SMD:C_0603_1608Metric_Pad1.08x0.95mm_HandSolder
- C405: renamed from C27; footprint (none) -> Capacitor_SMD:C_0603_1608Metric_Pad1.08x0.95mm_HandSolder
- C406: renamed from C28; footprint (none) -> Capacitor_SMD:C_0603_1608Metric_Pad1.08x0.95mm_HandSolder
- C407: renamed from C29; footprint (none) -> Capacitor_SMD:C_0603_1608Metric_Pad1.08x0.95mm_HandSolder
- C408: renamed from C47; footprint (none) -> Capacitor_SMD:C_0603_1608Metric_Pad1.08x0.95mm_HandSolder
- C409: renamed from C51; footprint (none) -> Capacitor_SMD:C_0603_1608Metric_Pad1.08x0.95mm_HandSolder
- C410: renamed from C59; footprint (none) -> Capacitor_SMD:C_0603_1608Metric_Pad1.08x0.95mm_HandSolder
- C411: renamed from C61; footprint (none) -> Capacitor_SMD:C_0603_1608Metric_Pad1.08x0.95mm_HandSolder
- C412: renamed from C60; footprint (none) -> Capacitor_SMD:C_0603_1608Metric_Pad1.08x0.95mm_HandSolder
- C413: renamed from C62; footprint (none) -> Capacitor_SMD:C_0603_1608Metric_Pad1.08x0.95mm_HandSolder
- C414: renamed from C601; footprint (none) -> Capacitor_SMD:C_0603_1608Metric_Pad1.08x0.95mm_HandSolder
- C415: renamed from C43; footprint (none) -> Capacitor_SMD:C_0603_1608Metric_Pad1.08x0.95mm_HandSolder
- C416: renamed from C58; footprint (none) -> Capacitor_SMD:C_0603_1608Metric_Pad1.08x0.95mm_HandSolder
- C417: renamed from C63; footprint (none) -> Capacitor_SMD:C_0603_1608Metric_Pad1.08x0.95mm_HandSolder
- C418: renamed from C602; footprint (none) -> Capacitor_SMD:C_0603_1608Metric_Pad1.08x0.95mm_HandSolder
- C419: renamed from C44; footprint (none) -> Capacitor_SMD:C_0603_1608Metric_Pad1.08x0.95mm_HandSolder
- C420: renamed from C603; footprint (none) -> Capacitor_SMD:C_0603_1608Metric_Pad1.08x0.95mm_HandSolder
- C421: renamed from C18; footprint (none) -> Capacitor_SMD:C_0603_1608Metric_Pad1.08x0.95mm_HandSolder
- C422: renamed from C42; footprint (none) -> Capacitor_SMD:C_0603_1608Metric_Pad1.08x0.95mm_HandSolder
- C423: renamed from C604; footprint (none) -> Capacitor_SMD:C_0603_1608Metric_Pad1.08x0.95mm_HandSolder
- C424: renamed from C40; footprint (none) -> Capacitor_SMD:C_0603_1608Metric_Pad1.08x0.95mm_HandSolder
- C425: renamed from C605; footprint (none) -> Capacitor_SMD:C_0603_1608Metric_Pad1.08x0.95mm_HandSolder
- C426: renamed from C41; footprint (none) -> Capacitor_SMD:C_0603_1608Metric_Pad1.08x0.95mm_HandSolder
- C427: renamed from C606; footprint (none) -> Capacitor_SMD:C_0603_1608Metric_Pad1.08x0.95mm_HandSolder
- C428: renamed from C33; footprint (none) -> Capacitor_SMD:C_0603_1608Metric_Pad1.08x0.95mm_HandSolder
- C429: renamed from C32; footprint (none) -> Capacitor_SMD:C_0603_1608Metric_Pad1.08x0.95mm_HandSolder
- C430: renamed from C49; footprint (none) -> Capacitor_SMD:C_0603_1608Metric_Pad1.08x0.95mm_HandSolder
- C431: renamed from C50; footprint (none) -> Capacitor_SMD:C_0603_1608Metric_Pad1.08x0.95mm_HandSolder
- FB401: renamed from FB2; footprint (none) -> Inductor_SMD:L_0603_1608Metric_Pad1.05x0.95mm_HandSolder
- FB402: renamed from FB1; footprint (none) -> Inductor_SMD:L_0603_1608Metric_Pad1.05x0.95mm_HandSolder
- J401: renamed from J4; footprint (none) -> Connector_Coaxial:SMA_Amphenol_901-144_Vertical
- J402: renamed from J8; footprint (none) -> Connector_Coaxial:SMA_Amphenol_901-144_Vertical
- J403: renamed from J2; footprint (none) -> Connector_Coaxial:SMA_Amphenol_901-144_Vertical
- R401: renamed from R8; footprint (none) -> Resistor_SMD:R_0603_1608Metric_Pad0.98x0.95mm_HandSolder
- R402: renamed from R28; footprint (none) -> Resistor_SMD:R_0603_1608Metric_Pad0.98x0.95mm_HandSolder
- R403: renamed from R27; footprint (none) -> Resistor_SMD:R_0603_1608Metric_Pad0.98x0.95mm_HandSolder
- R404: renamed from R57; footprint (none) -> Resistor_SMD:R_0603_1608Metric_Pad0.98x0.95mm_HandSolder
- R405: renamed from R26; footprint (none) -> Resistor_SMD:R_0603_1608Metric_Pad0.98x0.95mm_HandSolder
- R406: renamed from R58; footprint (none) -> Resistor_SMD:R_0603_1608Metric_Pad0.98x0.95mm_HandSolder
- R407: renamed from R25; footprint (none) -> Resistor_SMD:R_0603_1608Metric_Pad0.98x0.95mm_HandSolder
- R408: renamed from R59; footprint (none) -> Resistor_SMD:R_0603_1608Metric_Pad0.98x0.95mm_HandSolder
- R409: renamed from R5; footprint (none) -> Resistor_SMD:R_0603_1608Metric_Pad0.98x0.95mm_HandSolder
- R410: renamed from R34; footprint (none) -> Resistor_SMD:R_0603_1608Metric_Pad0.98x0.95mm_HandSolder
- R411: renamed from R31; footprint (none) -> Resistor_SMD:R_0603_1608Metric_Pad0.98x0.95mm_HandSolder
- R412: renamed from R35; footprint (none) -> Resistor_SMD:R_0603_1608Metric_Pad0.98x0.95mm_HandSolder
- R413: renamed from R32; footprint (none) -> Resistor_SMD:R_0603_1608Metric_Pad0.98x0.95mm_HandSolder
- R414: renamed from R36; footprint (none) -> Resistor_SMD:R_0603_1608Metric_Pad0.98x0.95mm_HandSolder
- R415: renamed from R33; footprint (none) -> Resistor_SMD:R_0603_1608Metric_Pad0.98x0.95mm_HandSolder
- R416: renamed from R37; footprint (none) -> Resistor_SMD:R_0603_1608Metric_Pad0.98x0.95mm_HandSolder
- R417: renamed from R30; footprint (none) -> Resistor_SMD:R_0603_1608Metric_Pad0.98x0.95mm_HandSolder
- SW401: renamed from SW2; footprint (none) -> Button_Switch_THT:SW_Slide_SPDT_Straight_CK_OS102011MS2Q
- SW402: renamed from SW4; footprint (none) -> Button_Switch_THT:SW_Slide_SPDT_Straight_CK_OS102011MS2Q
- SW403: renamed from SW5; footprint (none) -> Button_Switch_THT:SW_Slide_SPDT_Straight_CK_OS102011MS2Q
- TP401: renamed from TP2; footprint (none) -> TestPoint:TestPoint_Pad_D4.0mm
- TP402: renamed from TP3; footprint (none) -> TestPoint:TestPoint_Pad_D4.0mm
- TP403: renamed from TP1; footprint (none) -> TestPoint:TestPoint_Pad_D4.0mm
- U401: renamed from U4; footprint SO-8_S_LIT -> NonKiCad_footprints:SO-8_S_LIT-L
- U402: renamed from U5; footprint SO-8_S_LIT -> NonKiCad_footprints:SO-8_S_LIT-L
- U403: renamed from U3; footprint ST_64_1_ADI -> NonKiCad_footprints:ST_64_1_ADI
- U404: renamed from U8; footprint R_8_ADI -> NonKiCad_footprints:R_8_ADI
- U405: renamed from U7; footprint R_8_ADI -> NonKiCad_footprints:R_8_ADI

Commit message: Layout
Layout
Parts:
- removed TP401, TP402, TP403: TestPoint, TestPoint:TestPoint_Pad_D4.0mm, symbol Connector:TestPoint
Connections:
- net VREF_ADCD: now also C415.1, C419.1, U403.8 (VREF)
Changed lines of the file:
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@@
 	)
 	(junction
-		(at 179.07 147.32)
-		(diameter 0)
-		(color 0 0 0 0)
-	)
-	(junction
-		(at 154.94 146.05)
-		(diameter 0)
-		(color 0 0 0 0)
-	)
-	(junction
 		(at 237.49 223.52)
 		(diameter 0)
@@
 	)
 	(junction
-		(at 213.36 227.33)
-		(diameter 0)
-		(color 0 0 0 0)
-	)
-	(junction
 		(at 241.3 140.97)
 		(diameter 0)
@@
 	(wire
 		(pts
-			(xy 154.94 146.05) (xy 154.94 153.67)
+			(xy 154.94 133.35) (xy 154.94 153.67)
 		)
 		(stroke
@@
 	(wire
 		(pts
-			(xy 154.94 133.35) (xy 154.94 146.05)
-		)
-		(stroke
-			(width 0)
-			(type default)
-		)
-	)
-	(wire
-		(pts
 			(xy 195.58 219.71) (xy 219.71 219.71)
 		)
@@
 	(wire
 		(pts
-			(xy 179.07 133.35) (xy 179.07 147.32)
-		)
-		(stroke
-			(width 0)
-			(type default)
-		)
-	)
-	(wire
-		(pts
 			(xy 248.92 207.01) (xy 248.92 210.82)
 		)
@@
 	(wire
 		(pts
-			(xy 179.07 147.32) (xy 179.07 153.67)
+			(xy 179.07 133.35) (xy 179.07 153.67)
 		)
 		(stroke
@@
 		)
 	)
+	(global_label "VREF_ADCD"
+		(shape input)
+		(at 213.36 236.22 0)
+		(fields_autoplaced yes)
+		(effects
+			(font
+				(size 1.27 1.27)
+			)
+			(justify left)
+		)
+		(property "Intersheetrefs" "${INTERSHEET_REFS}"
+			(at 226.8076 236.22 0)
+			(effects
+				(font
+					(size 1.27 1.27)
+				)
+				(justify left)
+				(hide yes)
+			)
+		)
+	)
 	(global_label "clk_a_adc"
 		(shape input)
@@
 	)
 	(symbol
-		(lib_id "Connector:TestPoint")
-		(at 213.36 227.33 270)
-		(unit 1)
-		(exclude_from_sim no)
-		(in_bom yes)
-		(on_board yes)
-		(dnp no)
-		(fields_autoplaced yes)
-		(property "Reference" "TP403"
-			(at 218.44 226.0599 90)
-			(effects
-				(font
-					(size 1.27 1.27)
-				)
-				(justify left)
-			)
-		)
-		(property "Value" "TestPoint"
-			(at 218.44 228.5999 90)
-			(effects
-				(font
-					(size 1.27 1.27)
-				)
-				(justify left)
-				(hide yes)
-			)
-		)
-		(property "Footprint" "TestPoint:TestPoint_Pad_D4.0mm"
-			(at 213.36 232.41 0)
-			(effects
-				(font
-					(size 1.27 1.27)
-				)
-				(hide yes)
-			)
-		)
-		(property "Datasheet" "~"
-			(at 213.36 232.41 0)
-			(effects
-				(font
-					(size 1.27 1.27)
-				)
-				(hide yes)
-			)
-		)
-		(property "Description" "test point"
-			(at 213.36 227.33 0)
-			(effects
-				(font
-					(size 1.27 1.27)
-				)
-				(hide yes)
-			)
-		)
-		(pin "1"
-		)
-		(instances
-			(project "VNA_Project"
-				(path "/8b9c6944-c5f7-4a92-a452-dc4fa5f3924d/e352f3b5-433e-42a1-adc5-ff1237016ad8"
-					(reference "TP403")
-					(unit 1)
-				)
-			)
-		)
-	)
-	(symbol
 		(lib_id "Device:C_Small")
 		(at 283.21 62.23 0)
@@
 	)
 	(symbol
-		(lib_id "Connector:TestPoint")
-		(at 154.94 146.05 270)
-		(unit 1)
-		(exclude_from_sim no)
-		(in_bom yes)
-		(on_board yes)
-		(dnp no)
-		(fields_autoplaced yes)
-		(property "Reference" "TP401"
-			(at 160.02 144.7799 90)
-			(effects
-				(font
-					(size 1.27 1.27)
-				)
-				(justify left)
-			)
-		)
-		(property "Value" "TestPoint"
-			(at 160.02 147.3199 90)
-			(effects
-				(font
-					(size 1.27 1.27)
-				)
-				(justify left)
-				(hide yes)
-			)
-		)
-		(property "Footprint" "TestPoint:TestPoint_Pad_D4.0mm"
-			(at 154.94 151.13 0)
-			(effects
-				(font
-					(size 1.27 1.27)
-				)
-				(hide yes)
-			)
-		)
-		(property "Datasheet" "~"
-			(at 154.94 151.13 0)
-			(effects
-				(font
-					(size 1.27 1.27)
-				)
-				(hide yes)
-			)
-		)
-		(property "Description" "test point"
-			(at 154.94 146.05 0)
-			(effects
-				(font
-					(size 1.27 1.27)
-				)
-				(hide yes)
-			)
-		)
-		(pin "1"
-		)
-		(instances
-			(project "VNA_Project"
-				(path "/8b9c6944-c5f7-4a92-a452-dc4fa5f3924d/e352f3b5-433e-42a1-adc5-ff1237016ad8"
-					(reference "TP401")
-					(unit 1)
-				)
-			)
-		)
-	)
-	(symbol
 		(lib_id "Device:C_Small")
 		(at 201.93 49.53 180)
@@
 					(unit 1)
 				)
-			)
-		)
-	)
-	(symbol
-		(lib_id "Connector:TestPoint")
-		(at 179.07 147.32 90)
-		(unit 1)
-		(exclude_from_sim no)
-		(in_bom yes)
-		(on_board yes)
-		(dnp no)
-		(fields_autoplaced yes)
-		(property "Reference" "TP402"
-			(at 175.768 144.78 90)
-			(effects
-				(font
-					(size 1.27 1.27)
-				)
-			)
-		)
-		(property "Value" "TestPoint"
-			(at 173.99 146.0501 90)
-			(effects
-				(font
-					(size 1.27 1.27)
-				)
-				(justify left)
-				(hide yes)
-			)
-		)
-		(property "Footprint" "TestPoint:TestPoint_Pad_D4.0mm"
-			(at 179.07 142.24 0)
-			(effects
-				(font
-					(size 1.27 1.27)
-				)
-				(hide yes)
-			)
-		)
-		(property "Datasheet" "~"
-			(at 179.07 142.24 0)
-			(effects
-				(font
-					(size 1.27 1.27)
-				)
-				(hide yes)
-			)
-		)
-		(property "Description" "test point"
-			(at 179.07 147.32 0)
-			(effects
-				(font
-					(size 1.27 1.27)
-				)
-				(hide yes)
-			)
-		)
-		(pin "1"
-		)
-		(instances
-			(project "VNA_Project"
-				(path "/8b9c6944-c5f7-4a92-a452-dc4fa5f3924d/e352f3b5-433e-42a1-adc5-ff1237016ad8"
-					(reference "TP402")
-					(unit 1)
-				)
