File: VNA_Project/Directional_Coupler.kicad_sch (KiCad schematic)
At the start: 0 parts

Commit message: finishing up front end
refining Non RF front end
Other:
- note added: "Dir coupler is finished in ADS, will be creating a separate board to connect via Coax to test each part separately"
Changed lines of the file:
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@@
 	(generator_version "9.0")
 	(paper "A4")
+	(text "Dir coupler is finished in ADS, will be creating a separate board to connect via Coax to test each part separately\n"
+		(exclude_from_sim no)
+		(at 72.644 17.272 0)
+		(effects
+			(font
+				(size 1.27 1.27)
+			)
+		)
+	)
 )

Commit message: footprints + initial layout shape
footprints + initial layout shape
Other:
- note added: "Dir coupler is being done in ADS, will be creating a separate board to connect via Coax to test each part separately"
- note removed: "Dir coupler is finished in ADS, will be creating a separate board to connect via Coax to test each part separately"
Changed lines of the file:
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@@
 	(generator_version "9.0")
 	(paper "A4")
-	(text "Dir coupler is finished in ADS, will be creating a separate board to connect via Coax to test each part separately\n"
+	(text "Dir coupler is being done in ADS, will be creating a separate board to connect via Coax to test each part separately\n"
 		(exclude_from_sim no)
 		(at 72.644 17.272 0)
