File: VNA_Project/Ethernet.kicad_sch (KiCad schematic)
At the start: 32 parts, among them J502 8P8C_LED_Shielded_x2, SW501 SW_SPDT, U501 LAN8742A, U502 USBLC6-4SC6, Y501 STDCZS1-25M

Commit message: layout
layout
Parts:
- removed L501: 600R @ 100 MHz, Inductor_SMD:L_0805_2012Metric_Pad1.15x1.40mm_HandSolder, symbol Device:L
- removed TP501, TP502: TestPoint, TestPoint:TestPoint_Pad_D4.0mm, symbol Connector:TestPoint
- added FB501: FerriteBead, Inductor_SMD:L_0603_1608Metric_Pad1.05x0.95mm_HandSolder, symbol Device:FerriteBead
Connections:
- net +3.3VA: now also FB501.1
- net CT: now also FB501.2
Changed lines of the file:
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@@
 	)
 	(junction
-		(at 128.27 41.91)
-		(diameter 0)
-		(color 0 0 0 0)
-	)
-	(junction
 		(at 134.62 36.83)
 		(diameter 0)
@@
 	)
 	(junction
-		(at 123.19 41.91)
-		(diameter 0)
-		(color 0 0 0 0)
-	)
-	(junction
 		(at 172.72 68.58)
 		(diameter 0)
@@
 	(wire
 		(pts
-			(xy 123.19 41.91) (xy 123.19 45.72)
+			(xy 123.19 35.56) (xy 123.19 45.72)
 		)
 		(stroke
@@
 	(wire
 		(pts
-			(xy 123.19 35.56) (xy 123.19 41.91)
-		)
-		(stroke
-			(width 0)
-			(type default)
-		)
-	)
-	(wire
-		(pts
 			(xy 74.93 93.98) (xy 66.04 93.98)
 		)
@@
 	(wire
 		(pts
-			(xy 128.27 36.83) (xy 128.27 41.91)
+			(xy 128.27 36.83) (xy 128.27 45.72)
 		)
 		(stroke
@@
 	(wire
 		(pts
-			(xy 128.27 41.91) (xy 128.27 45.72)
-		)
-		(stroke
-			(width 0)
-			(type default)
-		)
-	)
-	(wire
-		(pts
 			(xy 100.33 96.52) (xy 107.95 96.52)
 		)
@@
 	)
 	(symbol
-		(lib_id "Connector:TestPoint")
-		(at 128.27 41.91 270)
-		(unit 1)
-		(exclude_from_sim no)
-		(in_bom yes)
-		(on_board yes)
-		(dnp no)
-		(fields_autoplaced yes)
-		(property "Reference" "TP502"
-			(at 133.35 41.9099 90)
-			(effects
-				(font
-					(size 1.27 1.27)
-				)
-				(justify left)
-			)
-		)
-		(property "Value" "TestPoint"
-			(at 133.35 43.1799 90)
-			(effects
-				(font
-					(size 1.27 1.27)
-				)
-				(justify left)
-				(hide yes)
-			)
-		)
-		(property "Footprint" "TestPoint:TestPoint_Pad_D4.0mm"
-			(at 128.27 46.99 0)
-			(effects
-				(font
-					(size 1.27 1.27)
-				)
-				(hide yes)
-			)
-		)
-		(property "Datasheet" "~"
-			(at 128.27 46.99 0)
-			(effects
-				(font
-					(size 1.27 1.27)
-				)
-				(hide yes)
-			)
-		)
-		(property "Description" "test point"
-			(at 128.27 41.91 0)
-			(effects
-				(font
-					(size 1.27 1.27)
-				)
-				(hide yes)
-			)
-		)
-		(pin "1"
-		)
-		(instances
-			(project "VNA_Project"
-				(path "/8b9c6944-c5f7-4a92-a452-dc4fa5f3924d/76256ba9-bc22-4fd8-98b4-4441e825b7f8"
-					(reference "TP502")
-					(unit 1)
-				)
-			)
-		)
-	)
-	(symbol
 		(lib_id "Device:C")
 		(at 175.26 43.18 0)
@@
 	)
 	(symbol
-		(lib_id "Connector:TestPoint")
-		(at 123.19 41.91 90)
+		(lib_id "Device:C")
+		(at 182.88 111.76 0)
 		(unit 1)
 		(exclude_from_sim no)
@@
 		(dnp no)
 		(fields_autoplaced yes)
-		(property "Reference" "TP501"
-			(at 119.888 39.37 90)
+		(property "Reference" "C509"
+			(at 186.69 110.4899 0)
 			(effects
 				(font
 					(size 1.27 1.27)
 				)
+				(justify left)
 			)
 		)
-		(property "Value" "TestPoint"
-			(at 118.11 40.6401 90)
+		(property "Value" "100n"
+			(at 186.69 113.0299 0)
 			(effects
 				(font
@@
 				)
 				(justify left)
-				(hide yes)
 			)
 		)
-		(property "Footprint" "TestPoint:TestPoint_Pad_D4.0mm"
-			(at 123.19 36.83 0)
+		(property "Footprint" "Capacitor_SMD:C_0603_1608Metric_Pad1.08x0.95mm_HandSolder"
+			(at 183.8452 115.57 0)
 			(effects
 				(font
@@
 		)
 		(property "Datasheet" "~"
-			(at 123.19 36.83 0)
+			(at 182.88 111.76 0)
 			(effects
 				(font
@@
 			)
 		)
-		(property "Description" "test point"
-			(at 123.19 41.91 0)
+		(property "Description" "Unpolarized capacitor"
+			(at 182.88 111.76 0)
 			(effects
 				(font
@@
 		(pin "1"
 		)
+		(pin "2"
+		)
 		(instances
-			(project "VNA_Project"
+			(project ""
 				(path "/8b9c6944-c5f7-4a92-a452-dc4fa5f3924d/76256ba9-bc22-4fd8-98b4-4441e825b7f8"
-					(reference "TP501")
+					(reference "C509")
 					(unit 1)
 				)
@@
 	)
 	(symbol
-		(lib_id "Device:C")
-		(at 182.88 111.76 0)
+		(lib_id "power:GND")
+		(at 158.75 123.19 180)
 		(unit 1)
 		(exclude_from_sim no)
@@
 		(dnp no)
 		(fields_autoplaced yes)
-		(property "Reference" "C509"
-			(at 186.69 110.4899 0)
+		(property "Reference" "#PWR0520"
+			(at 158.75 116.84 0)
 			(effects
 				(font
 					(size 1.27 1.27)
 				)
-				(justify left)
+				(hide yes)
 			)
 		)
-		(property "Value" "100n"
-			(at 186.69 113.0299 0)
+		(property "Value" "GND"
+			(at 158.75 118.11 0)
 			(effects
 				(font
 					(size 1.27 1.27)
 				)
-				(justify left)
+				(hide yes)
 			)
 		)
-		(property "Footprint" "Capacitor_SMD:C_0603_1608Metric_Pad1.08x0.95mm_HandSolder"
-			(at 183.8452 115.57 0)
+		(property "Footprint" ""
+			(at 158.75 123.19 0)
 			(effects
 				(font
@@
 			)
 		)
-		(property "Datasheet" "~"
-			(at 182.88 111.76 0)
+		(property "Datasheet" ""
+			(at 158.75 123.19 0)
 			(effects
 				(font
@@
 			)
 		)
-		(property "Description" "Unpolarized capacitor"
-			(at 182.88 111.76 0)
+		(property "Description" "Power symbol creates a global label with name \"GND\" , ground"
+			(at 158.75 123.19 0)
 			(effects
 				(font
@@
 		(pin "1"
 		)
-		(pin "2"
-		)
 		(instances
-			(project ""
+			(project "VNA_Project"
 				(path "/8b9c6944-c5f7-4a92-a452-dc4fa5f3924d/76256ba9-bc22-4fd8-98b4-4441e825b7f8"
-					(reference "C509")
+					(reference "#PWR0520")
 					(unit 1)
 				)
@@
 	)
 	(symbol
-		(lib_id "power:GND")
-		(at 158.75 123.19 180)
+		(lib_id "Device:FerriteBead")
+		(at 161.29 27.94 0)
 		(unit 1)
 		(exclude_from_sim no)
@@
 		(dnp no)
 		(fields_autoplaced yes)
-		(property "Reference" "#PWR0520"
-			(at 158.75 116.84 0)
+		(property "Reference" "FB501"
+			(at 165.1 26.6191 0)
 			(effects
 				(font
 					(size 1.27 1.27)
 				)
-				(hide yes)
+				(justify left)
 			)
 		)
-		(property "Value" "GND"
-			(at 158.75 118.11 0)
+		(property "Value" "FerriteBead"
+			(at 165.1 29.1591 0)
 			(effects
 				(font
 					(size 1.27 1.27)
 				)
-				(hide yes)
+				(justify left)
 			)
 		)
-		(property "Footprint" ""
-			(at 158.75 123.19 0)
+		(property "Footprint" "Inductor_SMD:L_0603_1608Metric_Pad1.05x0.95mm_HandSolder"
+			(at 159.512 27.94 90)
 			(effects
 				(font
@@
 			)
 		)
-		(property "Datasheet" ""
-			(at 158.75 123.19 0)
+		(property "Datasheet" "~"
+			(at 161.29 27.94 0)
 			(effects
 				(font
@@
 			)
 		)
-		(property "Description" "Power symbol creates a global label with name \"GND\" , ground"
-			(at 158.75 123.19 0)
+		(property "Description" "Ferrite bead"
+			(at 161.29 27.94 0)
 			(effects
 				(font
@@
 			)
 		)
+		(pin "2"
+		)
 		(pin "1"
 		)
 		(instances
-			(project "VNA_Project"
+			(project ""
 				(path "/8b9c6944-c5f7-4a92-a452-dc4fa5f3924d/76256ba9-bc22-4fd8-98b4-4441e825b7f8"
-					(reference "#PWR0520")
+					(reference "FB501")
 					(unit 1)
 				)
@@
 					(unit 1)
 				)
-			)
-		)
-	)
-	(symbol
-		(lib_id "Device:L")
-		(at 161.29 27.94 0)
-		(unit 1)
-		(exclude_from_sim no)
-		(in_bom yes)
-		(on_board yes)
-		(dnp no)
-		(fields_autoplaced yes)
-		(property "Reference" "L501"
-			(at 162.56 26.6699 0)
-			(effects
-				(font
-					(size 1.27 1.27)
-				)
-				(justify left)
-			)
-		)
-		(property "Value" "600R @ 100 MHz"
-			(at 162.56 29.2099 0)
-			(effects
-				(font
-					(size 1.27 1.27)
-				)
-				(justify left)
-			)
-		)
-		(property "Footprint" "Inductor_SMD:L_0805_2012Metric_Pad1.15x1.40mm_HandSolder"
-			(at 161.29 27.94 0)
-			(effects
-				(font
-					(size 1.27 1.27)
-				)
-				(hide yes)
-			)
-		)
-		(property "Datasheet" "~"
-			(at 161.29 27.94 0)
-			(effects
-				(font
-					(size 1.27 1.27)
-				)
-				(hide yes)
-			)
-		)
-		(property "Description" "Inductor"
-			(at 161.29 27.94 0)
-			(effects
-				(font
-					(size 1.27 1.27)
-				)
-				(hide yes)
-			)
-		)
-		(pin "2"
-		)
-		(pin "1"
-		)
-		(instances
-			(project ""
-				(path "/8b9c6944-c5f7-4a92-a452-dc4fa5f3924d/76256ba9-bc22-4fd8-98b4-4441e825b7f8"
-					(reference "L501")
-					(unit 1)
-				)
