File: VNA_Project/VNA_Project.kicad_pcb (KiCad board)
At the start: 2 copper layers, 200 x 200 mm, 1 part

Commit message: footprints + initial layout shape
footprints + initial layout shape
Parts:
- added C201: 10u, Capacitor_SMD:C_0805_2012Metric, F.Cu at (142.0, 144.2)
- added C202: 10uF, Capacitor_SMD:C_0805_2012Metric, F.Cu at (142.0, 147.2)
- added C203: 100n, Capacitor_SMD:C_0805_2012Metric, F.Cu at (142.0, 150.2)
- added C204: 100n, Capacitor_SMD:C_0805_2012Metric, F.Cu at (142.0, 153.2)
- added C205: 1u, Capacitor_SMD:C_0805_2012Metric, F.Cu at (142.0, 156.2)
- added C206: 100p, Capacitor_SMD:C_0805_2012Metric, F.Cu at (142.0, 159.2)
- added C207: 100nF, Capacitor_SMD:C_0805_2012Metric, F.Cu at (146.5, 144.2)
- added C208: 1u, Capacitor_SMD:C_0805_2012Metric, F.Cu at (146.5, 147.2)
- added C209: 22uF, Capacitor_SMD:C_0805_2012Metric, F.Cu at (146.5, 150.2)
- added C210: 22u, Capacitor_SMD:C_0805_2012Metric, F.Cu at (146.5, 153.2)
- added C211: 1u, Capacitor_SMD:C_0805_2012Metric, F.Cu at (146.5, 156.2)
- added C212: 22u, Capacitor_SMD:C_0805_2012Metric, F.Cu at (146.5, 159.2)
- added C213: 22uF, Capacitor_SMD:C_0805_2012Metric, F.Cu at (150.9, 144.2)
- added C214: 22u, Capacitor_SMD:C_0805_2012Metric, F.Cu at (150.9, 147.2)
- added C215: 22u, Capacitor_SMD:C_0805_2012Metric, F.Cu at (150.9, 150.2)
- added C216: 68u, Capacitor_SMD:C_0805_2012Metric, F.Cu at (150.9, 153.2)
- added C217: 1u, Capacitor_SMD:C_0805_2012Metric, F.Cu at (150.9, 156.2)
- added C218: 68u, Capacitor_SMD:C_0805_2012Metric, F.Cu at (150.9, 159.2)
- added C219: 68u, Capacitor_SMD:C_0805_2012Metric, F.Cu at (155.4, 144.2)
- added C220: 15u, Capacitor_SMD:C_0805_2012Metric, F.Cu at (155.4, 147.2)
- added C221: 0.1u, Capacitor_SMD:C_0805_2012Metric, F.Cu at (155.4, 150.2)
- added C222: 0.1u, Capacitor_SMD:C_0805_2012Metric, F.Cu at (155.4, 153.2)
- added C223: 1u, Capacitor_SMD:C_0805_2012Metric, F.Cu at (155.4, 156.2)
- added C224: 0.22u, Capacitor_SMD:C_0805_2012Metric, F.Cu at (155.4, 159.2)
- added C225: 0.01u, Capacitor_SMD:C_0805_2012Metric, F.Cu at (159.8, 144.2)
- added C226: DNF, Capacitor_SMD:C_0805_2012Metric, F.Cu at (159.8, 147.2)
- added C227: 1u, Capacitor_SMD:C_0805_2012Metric, F.Cu at (159.8, 150.2)
- added C228: 47u, Capacitor_SMD:C_0805_2012Metric, F.Cu at (159.8, 153.2)
- added C229: 47u, Capacitor_SMD:C_0805_2012Metric, F.Cu at (159.8, 156.2)
- added C230: 47u, Capacitor_SMD:C_0805_2012Metric, F.Cu at (159.8, 159.2)
- added C301: 10p, Capacitor_SMD:C_0603_1608Metric_Pad1.08x0.95mm_HandSolder, F.Cu at (142.0, 190.3)
- added C302: 1u, Capacitor_SMD:C_0603_1608Metric_Pad1.08x0.95mm_HandSolder, F.Cu at (142.0, 192.8)
- added C303: 4.7u, Capacitor_SMD:C_0603_1608Metric_Pad1.08x0.95mm_HandSolder, F.Cu at (142.0, 195.3)
- added C304: 10p, Capacitor_SMD:C_0603_1608Metric_Pad1.08x0.95mm_HandSolder, F.Cu at (142.0, 197.8)
- added C305: 100n, Capacitor_SMD:C_0603_1608Metric_Pad1.08x0.95mm_HandSolder, F.Cu at (142.0, 200.3)
- added C306: 100n, Capacitor_SMD:C_0603_1608Metric_Pad1.08x0.95mm_HandSolder, F.Cu at (142.0, 202.9)
- added C307: 100n, Capacitor_SMD:C_0603_1608Metric_Pad1.08x0.95mm_HandSolder, F.Cu at (142.0, 205.4)
- added C308: 100n, Capacitor_SMD:C_0603_1608Metric_Pad1.08x0.95mm_HandSolder, F.Cu at (142.0, 207.9)
- added C309: 100n, Capacitor_SMD:C_0603_1608Metric_Pad1.08x0.95mm_HandSolder, F.Cu at (142.0, 210.4)
- added C310: 100n, Capacitor_SMD:C_0603_1608Metric_Pad1.08x0.95mm_HandSolder, F.Cu at (146.3, 190.3)
- added C311: 100n, Capacitor_SMD:C_0603_1608Metric_Pad1.08x0.95mm_HandSolder, F.Cu at (146.3, 192.8)
- added C312: 100n, Capacitor_SMD:C_0603_1608Metric_Pad1.08x0.95mm_HandSolder, F.Cu at (146.3, 195.3)
- added C313: 100n, Capacitor_SMD:C_0603_1608Metric_Pad1.08x0.95mm_HandSolder, F.Cu at (146.3, 197.8)
- added C314: 1u, Capacitor_SMD:C_0603_1608Metric_Pad1.08x0.95mm_HandSolder, F.Cu at (146.3, 200.3)
- added C315: 100n, Capacitor_SMD:C_0603_1608Metric_Pad1.08x0.95mm_HandSolder, F.Cu at (146.3, 202.9)
- added C316: 100n, Capacitor_SMD:C_0603_1608Metric_Pad1.08x0.95mm_HandSolder, F.Cu at (146.3, 205.4)
- added C317: 100n, Capacitor_SMD:C_0603_1608Metric_Pad1.08x0.95mm_HandSolder, F.Cu at (146.3, 207.9)
- added C401: 10u, Capacitor_SMD:C_0603_1608Metric_Pad1.08x0.95mm_HandSolder, F.Cu at (100.3, 143.9)
- added C402: 0.1u, Capacitor_SMD:C_0603_1608Metric_Pad1.08x0.95mm_HandSolder, F.Cu at (100.3, 146.4)
- added C403: 100n, Capacitor_SMD:C_0603_1608Metric_Pad1.08x0.95mm_HandSolder, F.Cu at (100.3, 149.0)
- added C404: 100n, Capacitor_SMD:C_0603_1608Metric_Pad1.08x0.95mm_HandSolder, F.Cu at (100.3, 151.5)
- added C405: 0.1u, Capacitor_SMD:C_0603_1608Metric_Pad1.08x0.95mm_HandSolder, F.Cu at (100.3, 154.0)
- added C406: 0.1u, Capacitor_SMD:C_0603_1608Metric_Pad1.08x0.95mm_HandSolder, F.Cu at (100.3, 156.5)
- added C407: 0.1u, Capacitor_SMD:C_0603_1608Metric_Pad1.08x0.95mm_HandSolder, F.Cu at (100.3, 159.0)
- added C408: 100n, Capacitor_SMD:C_0603_1608Metric_Pad1.08x0.95mm_HandSolder, F.Cu at (100.3, 161.5)
- added C409: 100n, Capacitor_SMD:C_0603_1608Metric_Pad1.08x0.95mm_HandSolder, F.Cu at (100.3, 164.0)
- added C410: 12p, Capacitor_SMD:C_0603_1608Metric_Pad1.08x0.95mm_HandSolder, F.Cu at (100.3, 166.5)
- added C411: 12p, Capacitor_SMD:C_0603_1608Metric_Pad1.08x0.95mm_HandSolder, F.Cu at (100.3, 169.0)
- added C412: 100p, Capacitor_SMD:C_0603_1608Metric_Pad1.08x0.95mm_HandSolder, F.Cu at (104.6, 143.9)
- added C413: 100p, Capacitor_SMD:C_0603_1608Metric_Pad1.08x0.95mm_HandSolder, F.Cu at (104.6, 146.4)
- added C414: 0.1u, Capacitor_SMD:C_0603_1608Metric_Pad1.08x0.95mm_HandSolder, F.Cu at (104.6, 149.0)
- added C415: 0.1u, Capacitor_SMD:C_0603_1608Metric_Pad1.08x0.95mm_HandSolder, F.Cu at (104.6, 151.5)
- added C416: 100p, Capacitor_SMD:C_0603_1608Metric_Pad1.08x0.95mm_HandSolder, F.Cu at (104.6, 154.0)
- added C417: 100p, Capacitor_SMD:C_0603_1608Metric_Pad1.08x0.95mm_HandSolder, F.Cu at (104.6, 156.5)
- added C418: 0.1u, Capacitor_SMD:C_0603_1608Metric_Pad1.08x0.95mm_HandSolder, F.Cu at (104.6, 159.0)
- added C419: 10u, Capacitor_SMD:C_0603_1608Metric_Pad1.08x0.95mm_HandSolder, F.Cu at (104.6, 161.5)
- added C420: 0.1u, Capacitor_SMD:C_0603_1608Metric_Pad1.08x0.95mm_HandSolder, F.Cu at (104.6, 164.0)
- added C421: 0.1u, Capacitor_SMD:C_0603_1608Metric_Pad1.08x0.95mm_HandSolder, F.Cu at (104.6, 166.5)
- added C422: 0.1u, Capacitor_SMD:C_0603_1608Metric_Pad1.08x0.95mm_HandSolder, F.Cu at (104.6, 169.0)
- added C423: 10u, Capacitor_SMD:C_0603_1608Metric_Pad1.08x0.95mm_HandSolder, F.Cu at (109.0, 143.9)
- added C424: 0.1u, Capacitor_SMD:C_0603_1608Metric_Pad1.08x0.95mm_HandSolder, F.Cu at (109.0, 146.4)
- added C425: 10u, Capacitor_SMD:C_0603_1608Metric_Pad1.08x0.95mm_HandSolder, F.Cu at (109.0, 149.0)
- added C426: 10u, Capacitor_SMD:C_0603_1608Metric_Pad1.08x0.95mm_HandSolder, F.Cu at (109.0, 151.5)
- added C427: 10u, Capacitor_SMD:C_0603_1608Metric_Pad1.08x0.95mm_HandSolder, F.Cu at (109.0, 154.0)
- added C428: 100p, Capacitor_SMD:C_0603_1608Metric_Pad1.08x0.95mm_HandSolder, F.Cu at (109.0, 156.5)
- added C429: 100p, Capacitor_SMD:C_0603_1608Metric_Pad1.08x0.95mm_HandSolder, F.Cu at (109.0, 159.0)
- added C430: 100n, Capacitor_SMD:C_0603_1608Metric_Pad1.08x0.95mm_HandSolder, F.Cu at (109.0, 161.5)
- added C431: 100n, Capacitor_SMD:C_0603_1608Metric_Pad1.08x0.95mm_HandSolder, F.Cu at (109.0, 164.0)
- added C501: 10p, Capacitor_SMD:C_0603_1608Metric_Pad1.08x0.95mm_HandSolder, F.Cu at (120.2, 192.9)
- added C502: 10p, Capacitor_SMD:C_0603_1608Metric_Pad1.08x0.95mm_HandSolder, F.Cu at (120.2, 195.4)
- added C503: 100n, Capacitor_SMD:C_0603_1608Metric_Pad1.08x0.95mm_HandSolder, F.Cu at (120.2, 197.9)
- added C504: 1u, Capacitor_SMD:C_0603_1608Metric_Pad1.08x0.95mm_HandSolder, F.Cu at (120.2, 200.4)
- added C505: 470p, Capacitor_SMD:C_0603_1608Metric_Pad1.08x0.95mm_HandSolder, F.Cu at (120.2, 202.9)
- added C506: 100n, Capacitor_SMD:C_0603_1608Metric_Pad1.08x0.95mm_HandSolder, F.Cu at (120.2, 205.4)
- added C507: 100n, Capacitor_SMD:C_0603_1608Metric_Pad1.08x0.95mm_HandSolder, F.Cu at (120.2, 207.9)
- added C508: 10u, Capacitor_SMD:C_0603_1608Metric_Pad1.08x0.95mm_HandSolder, F.Cu at (120.2, 210.4)
- added C509: 100n, Capacitor_SMD:C_0603_1608Metric_Pad1.08x0.95mm_HandSolder, F.Cu at (124.6, 192.9)
- added C510: 100n, Capacitor_SMD:C_0603_1608Metric_Pad1.08x0.95mm_HandSolder, F.Cu at (124.6, 195.4)
- added C511: 100n, Capacitor_SMD:C_0603_1608Metric_Pad1.08x0.95mm_HandSolder, F.Cu at (124.6, 197.9)
- added D201: Green, LED_SMD:LED_0603_1608Metric_Pad1.05x0.95mm_HandSolder, F.Cu at (179.1, 172.2)
- added D202: Green, LED_SMD:LED_0603_1608Metric_Pad1.05x0.95mm_HandSolder, F.Cu at (179.1, 174.7)
- added D203: Green, LED_SMD:LED_0603_1608Metric_Pad1.05x0.95mm_HandSolder, F.Cu at (179.1, 177.3)
- added D204: Green, LED_SMD:LED_0603_1608Metric_Pad1.05x0.95mm_HandSolder, F.Cu at (179.1, 179.9)
- added D205: Green, LED_SMD:LED_0603_1608Metric_Pad1.05x0.95mm_HandSolder, F.Cu at (179.1, 182.5)
- added D206: Green, LED_SMD:LED_0603_1608Metric_Pad1.05x0.95mm_HandSolder, F.Cu at (179.1, 185.1)
- added D301: ESD131-B1-W0201, Diode_SMD:Infineon_SG-WLL-2-3_0.58x0.28_P0.36mm, F.Cu at (157.9, 212.6)
- added D302: ESD131-B1-W0201, Diode_SMD:Infineon_SG-WLL-2-3_0.58x0.28_P0.36mm, F.Cu at (157.9, 214.6)
- added D303: ESD131-B1-W0201, Diode_SMD:Infineon_SG-WLL-2-3_0.58x0.28_P0.36mm, F.Cu at (157.9, 216.5)
- added D304: ESD131-B1-W0201, Diode_SMD:Infineon_SG-WLL-2-3_0.58x0.28_P0.36mm, F.Cu at (157.9, 218.4)
- added D305: ESD131-B1-W0201, Diode_SMD:Infineon_SG-WLL-2-3_0.58x0.28_P0.36mm, F.Cu at (157.9, 220.4)
- added D306: RED, LED_SMD:LED_0603_1608Metric_Pad1.05x0.95mm_HandSolder, F.Cu at (142.0, 212.9)
- added D307: RED, LED_SMD:LED_0603_1608Metric_Pad1.05x0.95mm_HandSolder, F.Cu at (142.0, 215.5)
- added D308: RED, LED_SMD:LED_0603_1608Metric_Pad1.05x0.95mm_HandSolder, F.Cu at (142.0, 218.1)
- added D309: RED, LED_SMD:LED_0603_1608Metric_Pad1.05x0.95mm_HandSolder, F.Cu at (142.0, 220.7)
- added D310: RED, LED_SMD:LED_0603_1608Metric_Pad1.05x0.95mm_HandSolder, F.Cu at (142.0, 223.3)
- added FB301: FerriteBead, Inductor_SMD:L_0603_1608Metric_Pad1.05x0.95mm_HandSolder, F.Cu at (146.3, 210.4)
- added FB401: FerriteBead, Inductor_SMD:L_0603_1608Metric_Pad1.05x0.95mm_HandSolder, F.Cu at (109.0, 166.5)
- added FB402: FerriteBead, Inductor_SMD:L_0603_1608Metric_Pad1.05x0.95mm_HandSolder, F.Cu at (109.0, 169.0)
- added H301: MountingHole, MountingHole:MountingHole_2.2mm_M2, F.Cu at (200.7, 103.1)
- added H302: MountingHole, MountingHole:MountingHole_2.2mm_M2, F.Cu at (394.2, 102.7)
- added H303: MountingHole, MountingHole:MountingHole_2.2mm_M2, F.Cu at (394.0, 295.2)
- added H304: MountingHole, MountingHole:MountingHole_2.2mm_M2, F.Cu at (201.1, 294.4)
- added J201: USB_C_Receptacle_USB2.0_16P, Connector_USB:USB_C_Receptacle_G-Switch_GT-USB-7010ASV, F.Cu at (200.1, 229.6)
- added J202: Jack-DC, Connector_BarrelJack:BarrelJack_GCT_DCJ200-10-A_Horizontal, F.Cu at (205.7, 118.8)
- added J203: Screw_Terminal_01x01, TerminalBlock:TerminalBlock_MaiXu_MX126-5.0-02P_1x02_P5.00mm, F.Cu at (187.4, 205.4)
- added J301: 2x5 1.27mm, Connector_PinHeader_2.54mm:PinHeader_2x05_P2.54mm_Vertical, F.Cu at (172.4, 191.3)
- added J302: Screw_Terminal_01x02, TerminalBlock:TerminalBlock_MaiXu_MX126-5.0-02P_1x02_P5.00mm, F.Cu at (394.4, 198.7)
- added J401: Conn_Coaxial, Connector_Coaxial:SMA_Amphenol_901-144_Vertical, F.Cu at (124.6, 159.3)
- added J402: Conn_Coaxial, Connector_Coaxial:SMA_Amphenol_901-144_Vertical, F.Cu at (124.6, 168.7)
- added J403: Conn_Coaxial, Connector_Coaxial:SMA_Amphenol_901-144_Vertical, F.Cu at (124.6, 178.1)
- added J501: RJ45_Wuerth_7499010211A, Connector_RJ:RJ45_Wuerth_7499010211A_Horizontal, F.Cu at (210.8, 185.8)
- added L201: 10u, Inductor_SMD:L_0805_2012Metric_Pad1.15x1.40mm_HandSolder, F.Cu at (182.6, 144.2)
- added L202: 10n, Inductor_SMD:L_0805_2012Metric_Pad1.15x1.40mm_HandSolder, F.Cu at (182.6, 147.1)
- added L203: 3.9uH, Inductor_SMD:L_0805_2012Metric_Pad1.15x1.40mm_HandSolder, F.Cu at (182.6, 150.1)
- added L204: 10u, Inductor_SMD:L_0805_2012Metric_Pad1.15x1.40mm_HandSolder, F.Cu at (182.6, 153.0)
- added L501: 600R @ 100 MHz, Inductor_SMD:L_0805_2012Metric_Pad1.15x1.40mm_HandSolder, F.Cu at (112.9, 216.4)
- added LED301: CLMVC-FKA-CL1D1L71BB7C3C3, NonKiCad_footprints:CLMVC-FKA-CL1D1L71BB7C3C3_CRE, F.Cu at (131.6, 220.8)
- added R201: 5.1K, Resistor_SMD:R_0603_1608Metric_Pad0.98x0.95mm_HandSolder, F.Cu at (154.3, 162.0)
- added R202: 5.1K, Resistor_SMD:R_0603_1608Metric_Pad0.98x0.95mm_HandSolder, F.Cu at (154.3, 164.5)
- added R203: 1k, Resistor_SMD:R_0603_1608Metric_Pad0.98x0.95mm_HandSolder, F.Cu at (154.3, 167.0)
- added R204: 158k, Resistor_SMD:R_0603_1608Metric_Pad0.98x0.95mm_HandSolder, F.Cu at (154.3, 169.5)
- added R205: 30.1k, Resistor_SMD:R_0603_1608Metric_Pad0.98x0.95mm_HandSolder, F.Cu at (154.3, 172.0)
- added R206: 1k, Resistor_SMD:R_0603_1608Metric_Pad0.98x0.95mm_HandSolder, F.Cu at (158.7, 162.0)
- added R207: 1k, Resistor_SMD:R_0603_1608Metric_Pad0.98x0.95mm_HandSolder, F.Cu at (158.7, 164.5)
- added R208: 1k, Resistor_SMD:R_0603_1608Metric_Pad0.98x0.95mm_HandSolder, F.Cu at (158.7, 167.0)
- added R209: 1k, Resistor_SMD:R_0603_1608Metric_Pad0.98x0.95mm_HandSolder, F.Cu at (158.7, 169.5)
- added R210: 162k, Resistor_SMD:R_0603_1608Metric_Pad0.98x0.95mm_HandSolder, F.Cu at (158.7, 172.0)
- added R211: 1.54k, Resistor_SMD:R_0603_1608Metric_Pad0.98x0.95mm_HandSolder, F.Cu at (163.0, 162.0)
- added R212: 49.9, Resistor_SMD:R_0603_1608Metric_Pad0.98x0.95mm_HandSolder, F.Cu at (163.0, 164.5)
- added R213: 52.3k, Resistor_SMD:R_0603_1608Metric_Pad0.98x0.95mm_HandSolder, F.Cu at (163.0, 167.0)
- added R214: 10k, Resistor_SMD:R_0603_1608Metric_Pad0.98x0.95mm_HandSolder, F.Cu at (163.0, 169.5)
- added R215: 1k, Resistor_SMD:R_0603_1608Metric_Pad0.98x0.95mm_HandSolder, F.Cu at (163.0, 172.0)
- added R301: 1.5K, Resistor_SMD:R_0603_1608Metric_Pad0.98x0.95mm_HandSolder, F.Cu at (150.7, 190.3)
- added R302: 10k, Resistor_SMD:R_0603_1608Metric_Pad0.98x0.95mm_HandSolder, F.Cu at (150.7, 192.8)
- added R303: 1.5K, Resistor_SMD:R_0603_1608Metric_Pad0.98x0.95mm_HandSolder, F.Cu at (150.7, 195.3)
- added R304: 1.5K, Resistor_SMD:R_0603_1608Metric_Pad0.98x0.95mm_HandSolder, F.Cu at (150.7, 197.8)
- added R305: DNF, Resistor_SMD:R_0603_1608Metric_Pad0.98x0.95mm_HandSolder, F.Cu at (150.7, 200.3)
- added R306: 49R9, Resistor_SMD:R_0603_1608Metric_Pad0.98x0.95mm_HandSolder, F.Cu at (150.7, 202.9)
- added R307: 49R9, Resistor_SMD:R_0603_1608Metric_Pad0.98x0.95mm_HandSolder, F.Cu at (150.7, 205.4)
- added R308: 49R9, Resistor_SMD:R_0603_1608Metric_Pad0.98x0.95mm_HandSolder, F.Cu at (150.7, 207.9)
- added R309: 49R9, Resistor_SMD:R_0603_1608Metric_Pad0.98x0.95mm_HandSolder, F.Cu at (150.7, 210.4)
- added R310: 1.5K, Resistor_SMD:R_0603_1608Metric_Pad0.98x0.95mm_HandSolder, F.Cu at (155.0, 190.3)
- added R311: 1.5K, Resistor_SMD:R_0603_1608Metric_Pad0.98x0.95mm_HandSolder, F.Cu at (155.0, 192.8)
- added R312: 1.5K, Resistor_SMD:R_0603_1608Metric_Pad0.98x0.95mm_HandSolder, F.Cu at (155.0, 195.3)
- added R313: 47, Resistor_SMD:R_0603_1608Metric_Pad0.98x0.95mm_HandSolder, F.Cu at (155.0, 197.8)
- added R314: 1.5K, Resistor_SMD:R_0603_1608Metric_Pad0.98x0.95mm_HandSolder, F.Cu at (155.0, 200.3)
- added R315: 1.5K, Resistor_SMD:R_0603_1608Metric_Pad0.98x0.95mm_HandSolder, F.Cu at (155.0, 202.9)
- added R316: 1.5K, Resistor_SMD:R_0603_1608Metric_Pad0.98x0.95mm_HandSolder, F.Cu at (155.0, 205.4)
- added R317: 1000, Resistor_SMD:R_0603_1608Metric_Pad0.98x0.95mm_HandSolder, F.Cu at (155.0, 207.9)
- added R318: 1000, Resistor_SMD:R_0603_1608Metric_Pad0.98x0.95mm_HandSolder, F.Cu at (155.0, 210.4)
- added R319: 1k, Resistor_SMD:R_0603_1608Metric_Pad0.98x0.95mm_HandSolder, F.Cu at (159.4, 190.3)
- added R320: 1000, Resistor_SMD:R_0603_1608Metric_Pad0.98x0.95mm_HandSolder, F.Cu at (159.4, 192.8)
- added R321: 2k, Resistor_SMD:R_0603_1608Metric_Pad0.98x0.95mm_HandSolder, F.Cu at (159.4, 195.3)
- added R322: 1000, Resistor_SMD:R_0603_1608Metric_Pad0.98x0.95mm_HandSolder, F.Cu at (159.4, 197.8)
- added R323: 1000, Resistor_SMD:R_0603_1608Metric_Pad0.98x0.95mm_HandSolder, F.Cu at (159.4, 200.3)
- added R324: 1000, Resistor_SMD:R_0603_1608Metric_Pad0.98x0.95mm_HandSolder, F.Cu at (159.4, 202.9)
- added R325: 1000, Resistor_SMD:R_0603_1608Metric_Pad0.98x0.95mm_HandSolder, F.Cu at (159.4, 205.4)
- added R326: 1000, Resistor_SMD:R_0603_1608Metric_Pad0.98x0.95mm_HandSolder, F.Cu at (159.4, 207.9)
- added R401: 50, Resistor_SMD:R_0603_1608Metric_Pad0.98x0.95mm_HandSolder, F.Cu at (113.3, 143.9)
- added R402: 50, Resistor_SMD:R_0603_1608Metric_Pad0.98x0.95mm_HandSolder, F.Cu at (113.3, 146.4)
- added R403: 300, Resistor_SMD:R_0603_1608Metric_Pad0.98x0.95mm_HandSolder, F.Cu at (113.3, 149.0)
- added R404: 300, Resistor_SMD:R_0603_1608Metric_Pad0.98x0.95mm_HandSolder, F.Cu at (113.3, 151.5)
- added R405: 910, Resistor_SMD:R_0603_1608Metric_Pad0.98x0.95mm_HandSolder, F.Cu at (113.3, 154.0)
- added R406: 910, Resistor_SMD:R_0603_1608Metric_Pad0.98x0.95mm_HandSolder, F.Cu at (113.3, 156.5)
- added R407: 220, Resistor_SMD:R_0603_1608Metric_Pad0.98x0.95mm_HandSolder, F.Cu at (113.3, 159.0)
- added R408: 220, Resistor_SMD:R_0603_1608Metric_Pad0.98x0.95mm_HandSolder, F.Cu at (113.3, 161.5)
- added R409: 50, Resistor_SMD:R_0603_1608Metric_Pad0.98x0.95mm_HandSolder, F.Cu at (113.3, 164.0)
- added R410: 499, Resistor_SMD:R_0603_1608Metric_Pad0.98x0.95mm_HandSolder, F.Cu at (113.3, 166.5)
- added R411: 499, Resistor_SMD:R_0603_1608Metric_Pad0.98x0.95mm_HandSolder, F.Cu at (113.3, 169.0)
- added R412: 499, Resistor_SMD:R_0603_1608Metric_Pad0.98x0.95mm_HandSolder, F.Cu at (117.7, 143.9)
- added R413: 499, Resistor_SMD:R_0603_1608Metric_Pad0.98x0.95mm_HandSolder, F.Cu at (117.7, 146.4)
- added R414: 499, Resistor_SMD:R_0603_1608Metric_Pad0.98x0.95mm_HandSolder, F.Cu at (117.7, 149.0)
- added R415: 499, Resistor_SMD:R_0603_1608Metric_Pad0.98x0.95mm_HandSolder, F.Cu at (117.7, 151.5)
- added R416: 499, Resistor_SMD:R_0603_1608Metric_Pad0.98x0.95mm_HandSolder, F.Cu at (117.7, 154.0)
- added R417: 499, Resistor_SMD:R_0603_1608Metric_Pad0.98x0.95mm_HandSolder, F.Cu at (117.7, 156.5)
- added R501: 0, Resistor_SMD:R_0603_1608Metric_Pad0.98x0.95mm_HandSolder, F.Cu at (124.6, 200.4)
- added R502: 33, Resistor_SMD:R_0603_1608Metric_Pad0.98x0.95mm_HandSolder, F.Cu at (124.6, 202.9)
- added R503: 33, Resistor_SMD:R_0603_1608Metric_Pad0.98x0.95mm_HandSolder, F.Cu at (124.6, 205.4)
- added R504: 10k, Resistor_SMD:R_0603_1608Metric_Pad0.98x0.95mm_HandSolder, F.Cu at (124.6, 207.9)
- added R505: 12.1k, Resistor_SMD:R_0603_1608Metric_Pad0.98x0.95mm_HandSolder, F.Cu at (124.6, 210.4)
- added R506: 49.9, Resistor_SMD:R_0603_1608Metric_Pad0.98x0.95mm_HandSolder, F.Cu at (128.9, 192.9)
- added R507: 49.9, Resistor_SMD:R_0603_1608Metric_Pad0.98x0.95mm_HandSolder, F.Cu at (128.9, 195.4)
- added R508: 49.9, Resistor_SMD:R_0603_1608Metric_Pad0.98x0.95mm_HandSolder, F.Cu at (128.9, 197.9)
- added R509: 49.9, Resistor_SMD:R_0603_1608Metric_Pad0.98x0.95mm_HandSolder, F.Cu at (128.9, 200.4)
- added R510: 270, Resistor_SMD:R_0603_1608Metric_Pad0.98x0.95mm_HandSolder, F.Cu at (128.9, 202.9)
- added R511: 270, Resistor_SMD:R_0603_1608Metric_Pad0.98x0.95mm_HandSolder, F.Cu at (128.9, 205.4)
- added R512: 10K, Resistor_SMD:R_0603_1608Metric_Pad0.98x0.95mm_HandSolder, F.Cu at (128.9, 207.9)
- added SW201: SW_SPDT, Button_Switch_THT:SW_Slide_SPDT_Straight_CK_OS102011MS2Q, F.Cu at (156.1, 176.8)
- added SW202: SW_SPDT, Button_Switch_THT:SW_Slide_SPDT_Straight_CK_OS102011MS2Q, F.Cu at (156.1, 183.3)
- added SW301: SW_SPDT, Button_Switch_THT:SW_Slide_SPDT_Straight_CK_OS102011MS2Q, F.Cu at (148.2, 225.3)
- added SW401: SW_SPDT, Button_Switch_THT:SW_Slide_SPDT_Straight_CK_OS102011MS2Q, F.Cu at (312.2, 102.5)
- added SW402: SW_SPDT, Button_Switch_THT:SW_Slide_SPDT_Straight_CK_OS102011MS2Q, F.Cu at (325.0, 102.4)
- added SW403: SW_SPDT, Button_Switch_THT:SW_Slide_SPDT_Straight_CK_OS102011MS2Q, F.Cu at (337.8, 102.4)
- added TP201: TestPoint, TestPoint:TestPoint_Pad_D4.0mm, F.Cu at (165.1, 145.7)
- added TP202: TestPoint, TestPoint:TestPoint_Pad_D4.0mm, F.Cu at (165.1, 151.8)
- added TP203: TestPoint, TestPoint:TestPoint_Pad_D4.0mm, F.Cu at (171.1, 145.7)
- added TP204: TestPoint, TestPoint:TestPoint_Pad_D4.0mm, F.Cu at (171.1, 151.8)
- added TP205: TestPoint, TestPoint:TestPoint_Pad_D4.0mm, F.Cu at (177.2, 145.7)
- added TP206: TestPoint, TestPoint:TestPoint_Pad_D4.0mm, F.Cu at (177.2, 151.8)
- added TP401: TestPoint, TestPoint:TestPoint_Pad_D4.0mm, F.Cu at (113.1, 173.3)
- added TP402: TestPoint, TestPoint:TestPoint_Pad_D4.0mm, F.Cu at (113.1, 179.4)
- added TP403: TestPoint, TestPoint:TestPoint_Pad_D4.0mm, F.Cu at (113.1, 185.4)
- added TP501: TestPoint, TestPoint:TestPoint_Pad_D4.0mm, F.Cu at (101.1, 217.9)
- added TP502: TestPoint, TestPoint:TestPoint_Pad_D4.0mm, F.Cu at (101.1, 224.0)
- added TR501: Wuerth_749013011A, Transformer_SMD:Transformer_Ethernet_Wuerth_749013011A, F.Cu at (236.8, 191.2)
- added U201: AP63205WU, Package_TO_SOT_SMD:TSOT-23-6_HandSoldering, F.Cu at (181.3, 163.1)
- added U202: AP63203WU, Package_TO_SOT_SMD:TSOT-23-6_HandSoldering, F.Cu at (181.3, 167.7)
- added U203: USBLC6-2SC6, Package_TO_SOT_SMD:SOT-23-6_Handsoldering, F.Cu at (165.0, 157.2)
- added U204: HT7533-1, Package_TO_SOT_SMD:SOT-89-3_Handsoldering, F.Cu at (169.6, 184.0)
- added U205: MIC5501-3.0YM5, Package_TO_SOT_SMD:SOT-23-5_HandSoldering, F.Cu at (142.7, 179.9)
- added U206: TPS54620RGYR, NonKiCad_footprints:TPS54620RGYR, F.Cu at (149.0, 180.4)
- added U207: MCP1804x-A002xOT, Package_TO_SOT_SMD:SOT-23-5_HandSoldering, F.Cu at (142.7, 184.7)
- added U301: TMP75AID, NonKiCad_footprints:TMP75AID, F.Cu at (165.9, 192.4)
- added U302: TMP75AID, NonKiCad_footprints:TMP75AID, F.Cu at (165.9, 199.1)
- added U303: STM32H730VBTx, Package_QFP:LQFP-100_14x14mm_P0.5mm, F.Cu at (299.2, 189.9)
- added U304: TMP75AID, NonKiCad_footprints:TMP75AID, F.Cu at (165.9, 205.7)
- added U305: TL972IPWR, NonKiCad_footprints:TL972IPWR, F.Cu at (174.6, 206.2)
- added U401: LT1813CS8-TRPBF, NonKiCad_footprints:SO-8_S_LIT-L, F.Cu at (133.2, 171.1)
- added U402: LT1813CS8-TRPBF, NonKiCad_footprints:SO-8_S_LIT-L, F.Cu at (133.2, 177.5)
- added U403: AD9238BSTZ-20, NonKiCad_footprints:ST_64_1_ADI, F.Cu at (341.7, 190.7)
- added U404: AD8138ARZ, NonKiCad_footprints:R_8_ADI, F.Cu at (133.5, 157.9)
- added U405: AD8138ARZ, NonKiCad_footprints:R_8_ADI, F.Cu at (133.5, 164.6)
- added U501: LAN8742A, Package_DFN_QFN:VQFN-24-1EP_4x4mm_P0.5mm_EP2.5x2.5mm, F.Cu at (107.3, 218.1)
- added U502: USBLC6-4SC6, Package_TO_SOT_SMD:SOT-23-6_Handsoldering, F.Cu at (107.1, 223.7)
- added Y301: STDCZS1-25M, Crystal:Crystal_SMD_2016-4Pin_2.0x1.6mm, F.Cu at (278.8, 191.1)
- added Y501: STDCZS1-25M, Crystal:Crystal_SMD_2016-4Pin_2.0x1.6mm, F.Cu at (122.9, 220.6)
Other:
- outline, holes or cut-outs redrawn

Commit message: Layout
Layout
Parts:
- removed J501: RJ45_Wuerth_7499010211A, Connector_RJ:RJ45_Wuerth_7499010211A_Horizontal
- added J502: 8P8C_LED_Shielded_x2, Connector_RJ:RJ45_Wuerth_7499010211A_Horizontal, F.Cu at (215.1, 187.7)
- added R513: 270, Resistor_SMD:R_0603_1608Metric_Pad0.98x0.95mm_HandSolder, F.Cu at (94.5, 233.6)
- added R514: 270, Resistor_SMD:R_0603_1608Metric_Pad0.98x0.95mm_HandSolder, F.Cu at (94.5, 236.1)
- added R515: 10K, Resistor_SMD:R_0603_1608Metric_Pad0.98x0.95mm_HandSolder, F.Cu at (94.5, 238.6)
- added SW501: SW_SPDT, Button_Switch_THT:SW_Slide_SPDT_Straight_CK_OS102011MS2Q, F.Cu at (201.4, 209.4)
- H301, H302, H303, H304: footprint MountingHole:MountingHole_2.2mm_M2 -> MountingHole:MountingHole_5mm
- L201, L202, L203, L204: footprint Inductor_SMD:L_0805_2012Metric_Pad1.15x1.40mm_HandSolder -> Inductor_SMD:L_Bourns_SDR0604
- moved J402 268.8 mm to (392.0, 196.1)
- moved J401 267.8 mm to (391.6, 180.6)
- moved J403 248.0 mm to (343.8, 294.1)
- moved U402 246.0 mm to (378.5, 196.1), turned to 180 degrees
- moved U401 245.5 mm to (378.6, 179.6), turned to 180 degrees
- moved U404 231.8 mm to (362.1, 196.7)
- moved U405 229.0 mm to (362.0, 179.8)
- moved R319 178.6 mm to (311.2, 284.4), turned to 180 degrees
- moved R321 172.2 mm to (306.8, 284.4), turned to 180 degrees
- moved C317 171.4 mm to (303.6, 276.1), turned to 180 degrees
- moved C303 169.6 mm to (311.6, 199.1), turned to -90 degrees
- moved R316 169.0 mm to (324.0, 200.2)
- moved R315 169.0 mm to (323.9, 198.6)
- moved R314 168.9 mm to (323.9, 196.9)
- moved C309 164.9 mm to (306.5, 198.9), turned to -90 degrees
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Routing:
- net Net-(SW201-B): track 0.00 -> 126.6 mm, vias 0 -> 2
- net +5V: track 0.00 -> 77.5 mm, vias 0 -> 2
- net GND: track 0.00 -> 30.4 mm, vias 0 -> 29
- net +3.3V: track 0.00 -> 19.9 mm, vias 0 -> 3
- net +15V: track 0.00 -> 19.2 mm, vias 0 -> 2
- net /Power/5_volt_filt: track 0.00 -> 13.4 mm
- net Net-(U202-SW): track 0.00 -> 9.10 mm
- net Net-(U201-FB): track 0.00 -> 8.71 mm
- net Net-(U201-SW): track 0.00 -> 8.44 mm
- net +3.3VA: track 0.00 -> 3.52 mm
- net +3V0: track 0.00 -> 2.65 mm
- net Net-(U201-BST): track 0.00 -> 2.22 mm
- net Net-(U202-BST): track 0.00 -> 2.02 mm
- added copper zone on F.Cu, net +10V
- added copper zone on F.Cu, net +15V
- added copper zone on In2.Cu, net +3.3V
- added copper zone on F.Cu, net +5V
- added copper zone on F.Cu, net GND
- added copper zone on In1.Cu, net GND
- added copper zone on In4.Cu, net GND
Other:
- copper layers 2 -> 6
- board text added: "+10V"
- board text added: "+3.3V"
- board text added: "+3.3VA"
- board text added: "+3.3VDD"
- board text added: "+3V"
- board text added: "+3V for 2s complement GND for offset binary"
- board text added: "+5V"
- board text added: "-5V"
- board text added: "-5V not included"
- board text added: "0-9.9V"
- board text added: "10V"
- board text added: "15V IN"
- board text added: "5V"
- board text added: "ADC"
- board text added: "ADC CLK"
- board text added: "BOOT0"
- board text added: "CALIBRATION"
- board text added: "CLOCK"
- board text added: "DAC"
- board text added: "DEBUG LEDs"
- board text added: "DFS"
- board text added: "DOWNCONVERTER A Wave"
- board text added: "DOWNCONVERTER B Wave"
- board text added: "ETH"
- board text added: "ETH PIN 7"
- board text added: "GND"
- board text added: "GND NC"
- board text added: "Instrumentation"
- board text added: "NEGATIVE SUPPLY ENABLE"
- board text added: "NRST NC SWO SWCLK SWDIO"
- board text added: "OEB_A"
- board text added: "OEB_B"
- board text added: "Power Supply"
- board text added: "TEMP GRAD"
- board text added: "TVS"
- board text added: "USBC - FS"
- board text added: "VBUS"
- board text added: "VCO SWEEP OUT"

Commit message: layout
layout
Parts:
- removed L501: 600R @ 100 MHz, Inductor_SMD:L_0805_2012Metric_Pad1.15x1.40mm_HandSolder
- added FB501: FerriteBead, Inductor_SMD:L_0603_1608Metric_Pad1.05x0.95mm_HandSolder, F.Cu at (261.8, 232.1)
- H301, H302, H303, H304: footprint MountingHole:MountingHole_5mm -> MountingHole:MountingHole_2.2mm_M2
- L201, L202, L203, L204: footprint Inductor_SMD:L_Bourns_SDR0604 -> Inductor_SMD:L_APV_ANR6020
- moved C503 208.9 mm to (269.8, 234.4), turned to -45 degrees
- moved C504 205.5 mm to (266.4, 236.5)
- moved C505 204.8 mm to (266.5, 234.9)
- moved C507 203.0 mm to (266.8, 226.2), turned to 45 degrees
- moved C508 201.5 mm to (265.7, 225.0), turned to 45 degrees
- moved C506 197.9 mm to (260.7, 230.9), turned to -135 degrees
- moved C511 196.3 mm to (263.3, 224.0), turned to 135 degrees
- moved R501 196.2 mm to (261.1, 237.3), turned to -135 degrees
- moved R505 193.8 mm to (261.9, 228.6), turned to -45 degrees
- moved C228 191.4 mm to (296.5, 115.9), turned to -90 degrees
- moved C229 188.9 mm to (293.5, 115.9), turned to -90 degrees
- moved C230 186.4 mm to (290.4, 115.9), turned to -90 degrees
- moved C226 180.9 mm to (286.8, 117.2), turned to -90 degrees
- moved C225 179.9 mm to (286.4, 122.0), turned to -90 degrees
- moved C224 179.0 mm to (278.7, 117.3)
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Connections:
- net Net-(SW201-B) renamed /Power/SW_POWER
Routing:
- net LED_INTSEL: track 0.00 -> 77.7 mm, vias 0 -> 1
- net LED_REGOFF: track 0.00 -> 74.4 mm, vias 0 -> 1
- net -5V: track 0.24 -> 62.5 mm, vias 0 -> 4
- net EN_inverting: track 0.00 -> 36.1 mm
- net GND: track 30.4 -> 55.8 mm, vias 29 -> 51
- net Net-(U206-SS/TR): track 0.00 -> 17.4 mm, vias 0 -> 2
- net boot_inv: track 0.00 -> 15.4 mm
- net /Power/SW_POWER: track 126.6 -> 140.8 mm
- net vsns_inv: track 0.00 -> 13.7 mm
- net Net-(SW202-A): track 0.00 -> 13.6 mm
- net Net-(J203-Pin_1): track 0.00 -> 12.2 mm
- net /Ethernet/CT: track 0.00 -> 8.96 mm
- net /Ethernet/xtal2_eth: track 0.00 -> 7.19 mm
- net Net-(C226-Pad1): track 0.00 -> 5.89 mm
- net Net-(U501-XTAL1/CLKIN): track 0.00 -> 5.57 mm
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Other:
- board text added: "DNF"

Commit message: minor changes
minor changes
Parts:
- moved U403 6.60 mm to (345.5, 185.3)
- moved C305 4.67 mm to (283.6, 187.6)
- moved C307 4.51 mm to (283.7, 185.9)
- moved C304 3.71 mm to (276.6, 187.6)
- moved Y301 3.71 mm to (278.5, 190.3)
- moved C301 3.71 mm to (276.4, 193.2)
- moved C312 2.80 mm to (305.7, 203.9)
- moved C303 2.65 mm to (309.4, 200.6), turned to 45 degrees
- moved U401 2.00 mm to (379.8, 178.0)
- moved C413 2.00 mm to (110.5, 130.3)
- moved C416 2.00 mm to (110.5, 137.8)
- moved C419 2.00 mm to (110.5, 145.4)
- moved C422 2.00 mm to (110.5, 152.9)
- moved C424 2.00 mm to (114.8, 130.3)
- moved C427 2.00 mm to (114.8, 137.8)
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Routing:
- net NRST: track 0.00 -> 145.6 mm, vias 0 -> 3
- net GND: track 55.8 -> 103.6 mm, vias 51 -> 76
- net +3.3V: track 22.0 -> 61.1 mm, vias 3 -> 6
- net HSE_OUT: track 0.00 -> 15.7 mm
- net VCO_TUNE: track 0.00 -> 13.1 mm
- net /MCU/analog decoupling: track 0.00 -> 10.8 mm
- net /MCU/CONN_SWDIO: track 0.00 -> 10.6 mm
- net Net-(C304-Pad1): track 0.00 -> 9.66 mm
- net Net-(C310-Pad1): track 0.00 -> 9.30 mm
- net /MCU/CONN_SWCLK: track 0.00 -> 8.13 mm
- net /MCU/CONN_NRST: track 0.00 -> 8.09 mm
- net /MCU/CONN_SWO: track 0.00 -> 7.90 mm
- net Net-(U305-IN1-): track 0.00 -> 5.53 mm
- net Net-(SW301-B): track 0.00 -> 4.85 mm
- net HSE_IN: track 0.00 -> 3.82 mm
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
Commit message: minor changes
Minor Changes
Parts:
- moved R514 76.6 mm to (214.4, 180.1), turned to -90 degrees
- moved R515 75.7 mm to (211.0, 180.0), turned to -90 degrees
- moved R513 69.5 mm to (207.1, 179.9), turned to 90 degrees
- moved R313 32.1 mm to (286.8, 204.3), turned to 90 degrees
- moved TP501 21.7 mm to (107.1, 181.7)
- moved TP502 21.7 mm to (107.1, 187.8)
- moved TP402 13.0 mm to (107.1, 168.5)
- moved TP403 13.0 mm to (107.1, 174.5)
- moved TP401 12.8 mm to (107.2, 162.2)
- moved R315 5.87 mm to (327.9, 194.3)
- moved R314 5.87 mm to (327.9, 192.6)
- moved R316 5.87 mm to (327.9, 195.9)
- moved U304 5.87 mm to (334.7, 195.3)
- moved H303 5.70 mm to (394.3, 295.6)
- moved H302 5.23 mm to (394.3, 101.6)
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Routing:
- net debug_led5: track 0.00 -> 206.6 mm, vias 0 -> 2
- net debug_led7: track 0.00 -> 200.4 mm, vias 0 -> 2
- net debug_led8: track 0.00 -> 196.0 mm, vias 0 -> 2
- net debug_led6: track 0.00 -> 192.0 mm, vias 0 -> 2
- net debug_led1: track 0.00 -> 180.1 mm, vias 0 -> 2
- net debug_led3: track 0.00 -> 157.2 mm, vias 0 -> 2
- net debug_led4: track 0.00 -> 156.5 mm, vias 0 -> 2
- net debug_led2: track 0.00 -> 154.5 mm, vias 0 -> 2
- net BOOT0: track 0.00 -> 148.3 mm, vias 0 -> 2
- net DAC1_OUT: track 0.00 -> 146.7 mm, vias 0 -> 2
- net SWCLK: track 0.00 -> 140.5 mm, vias 0 -> 4
- net SWDIO: track 0.00 -> 132.5 mm, vias 0 -> 2
- net JTDO: track 0.00 -> 129.0 mm, vias 0 -> 2
- net I2C4_SDA: track 0.00 -> 79.3 mm, vias 0 -> 2
- net I2C4_SCL: track 0.00 -> 78.2 mm, vias 0 -> 2
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- added copper zone on In3.Cu, net GND

Commit message: Layout
Layout
Parts:
- moved C403 281.4 mm to (384.6, 174.9), turned to 180 degrees
- moved C404 280.4 mm to (377.6, 205.6), turned to -90 degrees
- moved R402 280.0 mm to (386.6, 213.3), turned to 90 degrees
- moved C416 277.9 mm to (385.1, 180.4)
- moved C417 274.7 mm to (378.6, 200.1)
- moved C413 274.6 mm to (374.8, 204.5), turned to 90 degrees
- moved R401 273.7 mm to (387.2, 183.1), turned to 90 degrees
- moved C408 272.1 mm to (375.7, 182.2), turned to 90 degrees
- moved C409 271.3 mm to (369.3, 213.8), turned to 90 degrees
- moved R408 270.7 mm to (383.3, 204.6), turned to -135 degrees
- moved C410 269.8 mm to (374.9, 173.9), turned to -90 degrees
- moved R406 269.2 mm to (381.4, 201.1), turned to 90 degrees
- moved R405 268.6 mm to (383.9, 183.6), turned to 45 degrees
- moved C412 268.4 mm to (374.0, 178.8), turned to 180 degrees
- moved C411 268.4 mm to (369.3, 205.6), turned to -90 degrees
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Connections:
- C415 pad 1: Net-(U403-VREF) -> VREF_ADCD
- C419 pad 1: Net-(U403-VREF) -> VREF_ADCD
- U403 pad 8: Net-(U403-VREF) -> VREF_ADCD
Routing:
- net I2C1_SDA: track 5.44 -> 224.3 mm, vias 0 -> 4
- net I2C1_SCL: track 5.40 -> 218.7 mm, vias 0 -> 4
- net GND: track 120.2 -> 219.7 mm, vias 108 -> 148
- net Net-(SW401-B): track 0.00 -> 89.1 mm, vias 0 -> 1
- net VREF_ADCD: track 0.00 -> 64.2 mm, vias 0 -> 4
- net clk_a_adc: track 0.00 -> 30.5 mm
- net OUTB: track 0.00 -> 22.4 mm
- net Net-(U403-REFT_A): track 0.00 -> 21.3 mm
- net Net-(C414-Pad1): track 0.00 -> 21.0 mm
- net Net-(C412-Pad2): track 0.00 -> 19.8 mm
- net diffout_-: track 0.00 -> 16.5 mm
- net OUTB2: track 0.00 -> 16.0 mm
- net Net-(U404--IN): track 0.00 -> 15.6 mm
- net Net-(J402-Ext): track 0.00 -> 15.1 mm
- net +3V0: track 2.65 -> 17.4 mm, vias 0 -> 2
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- added copper zone on F.Cu, net +3V0
Other:
- board text removed: "ADC CLK"
- board text removed: "Flatrim Dreshaj VNA I"
