File: VNA_Project/VNA_Project.kicad_pcb (KiCad board)
At the start: 6 copper layers, 200 x 200 mm, 241 parts, among them J201 USB_C_Receptacle_USB2.0_16P, J202 Jack-DC, J203 Screw_Terminal_01x01, J301 2x5 1.27mm, J302 Screw_Terminal_01x02, J401 Conn_Coaxial, J402 Conn_Coaxial, J403 Conn_Coaxial, J502 8P8C_LED_Shielded_x2, SW201 SW_SPDT, SW202 SW_SPDT, SW301 SW_SPDT, SW401 SW_SPDT, SW402 SW_SPDT, SW403 SW_SPDT, SW501 SW_SPDT, U201 AP63205WU, U202 AP63203WU, U203 USBLC6-2SC6, U204 HT7533-1, U205 MIC5501-3.0YM5, U206 TPS54620RGYR, U207 MCP1804x-A002xOT, U301 TMP75AID, U302 TMP75AID, U303 STM32H730VBTx, U304 TMP75AID, U305 TL972IPWR, U401 LT1813CS8-TRPBF, U402 LT1813CS8-TRPBF, U403 AD9238BSTZ-20, U404 AD8138ARZ, U405 AD8138ARZ, U501 LAN8742A, U502 USBLC6-4SC6, Y301 STDCZS1-25M, Y501 STDCZS1-25M

Commit message: ethernet Layout
Ethernet Layout
Parts:
- removed J502: 8P8C_LED_Shielded_x2, Connector_RJ:RJ45_Wuerth_7499010211A_Horizontal
- removed R513, R514: 270, Resistor_SMD:R_0603_1608Metric_Pad0.98x0.95mm_HandSolder
- removed R515: 10K, Resistor_SMD:R_0603_1608Metric_Pad0.98x0.95mm_HandSolder
- removed SW501: SW_SPDT, Button_Switch_THT:SW_Slide_SPDT_Straight_CK_OS102011MS2Q
- removed TP401, TP402, TP403, TP501, TP502: TestPoint, TestPoint:TestPoint_Pad_D4.0mm
- removed TR501: Wuerth_749013011A, Transformer_SMD:Transformer_Ethernet_Wuerth_749013011A
- added J501: RJ45_Amphenol_RJMG1BD3B8K1ANR, Connector_RJ:RJ45_Amphenol_RJMG1BD3B8K1ANR, F.Cu at (215.2, 187.4)
- C503, C510, R504: moved to B.Cu
- moved C422 246.4 mm to (354.4, 187.5)
- moved R502 165.8 mm to (289.5, 231.0)
- moved R504 148.5 mm to (272.0, 234.2), turned to -45 degrees
- moved C510 148.3 mm to (270.5, 226.2), turned to 45 degrees
- moved C502 148.3 mm to (260.9, 239.8), turned to -135 degrees
- moved R503 147.5 mm to (268.9, 238.4), turned to 135 degrees
- moved C509 147.5 mm to (269.2, 224.8), turned to 45 degrees
- moved C501 143.2 mm to (256.4, 235.1), turned to -135 degrees
- moved R506 133.9 mm to (260.3, 221.8), turned to 135 degrees
- moved R508 127.8 mm to (254.8, 223.7), turned to 45 degrees
- moved R507 126.8 mm to (255.5, 215.8), turned to -135 degrees
- moved R509 122.6 mm to (251.7, 218.9), turned to 45 degrees
- moved R511 79.5 mm to (212.3, 180.0)
- moved R512 73.3 mm to (206.0, 182.2)
- moved R510 69.5 mm to (201.3, 204.0), turned to -90 degrees
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Connections:
- C506 pad 1: /Ethernet/CT -> /Ethernet/CRD
- C507 pad 1: /Ethernet/CT -> /Ethernet/CRD
- C508 pad 1: /Ethernet/CT -> /Ethernet/CRD
- C509 pad 1: /Ethernet/CT -> /Ethernet/CRD
- C510 pad 1: /Ethernet/CT -> /Ethernet/CRD
- C511 pad 1: /Ethernet/CT -> /Ethernet/CRD
- FB501 pad 2: /Ethernet/CT -> /Ethernet/CRD
- R506 pad 1: /Ethernet/CT -> /Ethernet/CRD
- R506 pad 2: /Ethernet/TX+ -> TD+
- R507 pad 1: /Ethernet/CT -> /Ethernet/CRD
- R507 pad 2: /Ethernet/TX- -> TD-
- R508 pad 1: /Ethernet/CT -> /Ethernet/CRD
- R508 pad 2: /Ethernet/RX+ -> RD+
- R509 pad 1: /Ethernet/CT -> /Ethernet/CRD
- R509 pad 2: /Ethernet/RX- -> RD-
- U501 pad 1: /Ethernet/CT -> /Ethernet/CRD
- U501 pad 19: /Ethernet/CT -> /Ethernet/CRD
- U501 pad 20: /Ethernet/TX- -> TD-
- U501 pad 21: /Ethernet/TX+ -> TD+
- U501 pad 22: /Ethernet/RX- -> RD-
- U501 pad 23: /Ethernet/RX+ -> RD+
- U502 pad 1: /Ethernet/RX+ -> RD+
- U502 pad 3: /Ethernet/TX+ -> TD+
- U502 pad 4: /Ethernet/TX- -> TD-
- U502 pad 5: /Ethernet/CT -> /Ethernet/CRD
- U502 pad 6: /Ethernet/RX- -> RD-
Routing:
- net /Ethernet/CRD: track 0.00 -> 135.2 mm, vias 0 -> 7
- net TD-: track 0.00 -> 79.3 mm
- net TD+: track 0.00 -> 76.8 mm, vias 0 -> 2
- net RD+: track 0.00 -> 76.0 mm, vias 0 -> 1
- net RD-: track 0.00 -> 75.3 mm, vias 0 -> 3
- net ETH_RXD1: track 0.00 -> 57.6 mm
- net ETH_MDC: track 0.00 -> 52.7 mm
- net ETH_CRS_DV: track 0.00 -> 48.5 mm
- net ETH_MDIO: track 0.00 -> 46.9 mm
- net NRST: track 145.6 -> 126.7 mm, vias 3 -> 5
- net GND: track 219.7 -> 237.0 mm, vias 148 -> 186
- net ETH_RXD0: track 0.00 -> 14.1 mm
- net Net-(J501-PadL3): track 0.00 -> 10.7 mm
- net LED_INTSEL: track 77.7 -> 87.9 mm
- net /Ethernet/CT: track 8.96 -> 0.00 mm
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Other:
- board text removed: "ETH PIN 7"
- board text removed: "GND NC"

Commit message: minor changes
Minor changes
Parts:
- moved R502 17.4 mm to (273.2, 237.2), turned to -135 degrees
Routing:
- net ETH_RXD0: track 14.1 -> 49.2 mm
- net Net-(U501-RXD0/MODE0): track 0.00 -> 8.32 mm
- net GND: track 237.0 -> 240.5 mm, vias 186 -> 187
Changed lines of the file:
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@@
 	(footprint "Resistor_SMD:R_0603_1608Metric_Pad0.98x0.95mm_HandSolder"
 		(layer "F.Cu")
-		(at 289.451 231.003)
+		(at 273.161 237.237 -135)
 		(descr "Resistor SMD 0603 (1608 Metric), square (rectangular) end terminal, IPC-7351 nominal with elongated pad for handsoldering. (Body size source: IPC-SM-782 page 72, https://www.pcb-3d.com/wordpress/wp-content/uploads/ipc-sm-782a_amendment_1_and_2.pdf), generated with kicad-footprint-generator")
 		(tags "resistor handsolder")
 		(property "Reference" "R502"
-			(at 0 -1.43 0)
+			(at -3.80777 -0.086974 45)
 			(layer "F.SilkS")
 			(effects
@@
 		)
 		(property "Value" "33"
-			(at 0 1.43 0)
+			(at 0 1.43 45)
 			(layer "F.Fab")
 			(effects
@@
 		)
 		(property "Datasheet" "~"
-			(at 0 0 0)
+			(at 0 0 45)
 			(layer "F.Fab")
 			(hide yes)
@@
 		)
 		(property "Description" "Resistor, small symbol"
-			(at 0 0 0)
+			(at 0 0 45)
 			(layer "F.Fab")
 			(hide yes)
@@
 		(attr smd)
 		(fp_line
-			(start -0.254724 -0.5225)
-			(end 0.254724 -0.5225)
+			(start -0.254724 0.5225)
+			(end 0.254724 0.5225)
 			(stroke
 				(width 0.12)
@@
 		)
 		(fp_line
-			(start -0.254724 0.5225)
-			(end 0.254724 0.5225)
+			(start -0.254724 -0.5225)
+			(end 0.254724 -0.5225)
 			(stroke
 				(width 0.12)
@@
 		)
 		(fp_line
-			(start -1.65 -0.73)
-			(end 1.65 -0.73)
+			(start 1.65 0.73)
+			(end -1.65 0.73)
 			(stroke
 				(width 0.05)
@@
 		)
 		(fp_line
-			(start -1.65 0.73)
-			(end -1.65 -0.73)
+			(start 1.65 -0.73)
+			(end 1.65 0.73)
 			(stroke
 				(width 0.05)
@@
 		)
 		(fp_line
-			(start 1.65 -0.73)
-			(end 1.65 0.73)
+			(start -1.65 0.73)
+			(end -1.65 -0.73)
 			(stroke
 				(width 0.05)
@@
 		)
 		(fp_line
-			(start 1.65 0.73)
-			(end -1.65 0.73)
+			(start -1.65 -0.73)
+			(end 1.65 -0.73)
 			(stroke
 				(width 0.05)
@@
 		)
 		(fp_line
-			(start -0.8 -0.4125)
-			(end 0.8 -0.4125)
+			(start 0.8 0.4125)
+			(end -0.8 0.4125)
 			(stroke
 				(width 0.1)
@@
 		)
 		(fp_line
-			(start -0.8 0.4125)
-			(end -0.8 -0.4125)
+			(start 0.8 -0.4125)
+			(end 0.8 0.4125)
 			(stroke
 				(width 0.1)
@@
 		)
 		(fp_line
-			(start 0.8 -0.4125)
-			(end 0.8 0.4125)
+			(start -0.8 0.4125)
+			(end -0.8 -0.4125)
 			(stroke
 				(width 0.1)
@@
 		)
 		(fp_line
-			(start 0.8 0.4125)
-			(end -0.8 0.4125)
+			(start -0.8 -0.4125)
+			(end 0.8 -0.4125)
 			(stroke
 				(width 0.1)
@@
 		)
 		(fp_text user "${REFERENCE}"
-			(at 0 0 0)
+			(at 0 0 45)
 			(layer "F.Fab")
 			(effects
@@
 		)
 		(pad "1" smd roundrect
-			(at -0.9125 0)
+			(at -0.9125 0 225)
 			(size 0.975 0.95)
 			(layers "F.Cu" "F.Mask" "F.Paste")
@@
 		)
 		(pad "2" smd roundrect
-			(at 0.9125 0)
+			(at 0.9125 0 225)
 			(size 0.975 0.95)
 			(layers "F.Cu" "F.Mask" "F.Paste")
@@
 		(tags "capacitor handsolder")
 		(property "Reference" "C503"
-			(at 3.841863 -0.096249 135)
+			(at 1.37603 -3.999396 135)
 			(layer "B.SilkS")
 			(effects
@@
 		(tags "resistor handsolder")
 		(property "Reference" "R504"
-			(at 0.411536 -1.424113 135)
+			(at 0.568514 -4.221427 135)
 			(layer "B.SilkS")
 			(effects
@@
 	)
 	(via
+		(at 273.721 234.144)
+		(size 0.6)
+		(drill 0.3)
+		(layers "F.Cu" "B.Cu")
+		(net 1)
+	)
+	(via
 		(at 332.35 184.05)
 		(size 0.6)
@@
 	)
 	(segment
+		(start 272.981765 234.883235)
+		(end 273.721 234.144)
+		(width 0.5)
+		(layer "B.Cu")
+		(net 1)
+	)
+	(segment
+		(start 272.20659 235.36088)
+		(end 272.684235 234.883235)
+		(width 0.5)
+		(layer "B.Cu")
+		(net 1)
+	)
+	(segment
 		(start 272.019 224.802)
 		(end 271.24076 225.58024)
@@
 	)
 	(segment
+		(start 270.73388 235.36088)
+		(end 272.20659 235.36088)
+		(width 0.5)
+		(layer "B.Cu")
+		(net 1)
+	)
+	(segment
+		(start 272.684235 234.883235)
+		(end 272.981765 234.883235)
+		(width 0.5)
+		(layer "B.Cu")
+		(net 1)
+	)
+	(segment
 		(start 272.019 224.005)
 		(end 272.019 224.802)
@@
 	)
 	(segment
+		(start 267.802 234.989)
+		(end 270.695235 237.882235)
+		(width 0.355)
+		(layer "F.Cu")
+		(net 125)
+	)
+	(segment
+		(start 267.357257 232.765683)
+		(end 267.802 233.210426)
+		(width 0.2)
+		(layer "F.Cu")
+		(net 125)
+	)
+	(segment
+		(start 270.695235 237.882235)
+		(end 272.515765 237.882235)
+		(width 0.355)
+		(layer "F.Cu")
+		(net 125)
+	)
+	(segment
+		(start 267.802 233.210426)
+		(end 267.802 234.989)
+		(width 0.355)
+		(layer "F.Cu")
+		(net 125)
+	)
+	(segment
+		(start 273.806235 236.591765)
+		(end 278.137 232.261)
+		(width 0.355)
+		(layer "F.Cu")
+		(net 126)
+	)
+	(segment
 		(start 296.2035 209.6205)
 		(end 294.726 211.098)
-		(width 0.25)
+		(width 0.355)
+		(layer "F.Cu")
+		(net 126)
+	)
+	(segment
+		(start 279.748544 232.261)
+		(end 294.726 217.283544)
+		(width 0.355)
+		(layer "F.Cu")
+		(net 126)
+	)
+	(segment
+		(start 278.137 232.261)
+		(end 279.748544 232.261)
+		(width 0.355)
+		(layer "F.Cu")
+		(net 126)
+	)
+	(segment
+		(start 294.726 217.283544)
+		(end 294.726 211.098)
+		(width 0.355)
 		(layer "F.Cu")
 		(net 126)
@@
 		(start 296.2035 197.5785)
 		(end 296.2035 209.6205)
-		(width 0.25)
+		(width 0.355)
 		(layer "F.Cu")
 		(net 126)

Commit message: eth
eth
Routing:
- net USB_D-: track 0.00 -> 99.5 mm
- net USB_D+: track 0.00 -> 98.7 mm
- net ETH_TXD1: track 0.00 -> 53.7 mm, vias 0 -> 2
- net /Power/usbc_d+: track 0.00 -> 9.09 mm
- net /Power/usbc_d-: track 0.00 -> 9.03 mm
- net VBUS: track 11.4 -> 20.2 mm, vias 0 -> 2
- net diffout_-: track 16.5 -> 17.9 mm
- net diffout_+: track 8.14 -> 9.44 mm
- net /Power/CC_1_pulldown: track 6.52 -> 7.66 mm
- net /Power/CC_2_pulldown: track 6.74 -> 7.68 mm
- added copper zone on F.Cu, net USB_D+
- added copper zone on F.Cu, net USB_D-

Commit message: finished Routing
finished Routing
Parts:
- C431: moved to B.Cu
- moved C431 12.5 mm to (356.2, 175.2), turned to 180 degrees
- moved C312 0.82 mm to (304.9, 203.7)
Routing:
- net +5V: track 88.5 -> 446.0 mm, vias 2 -> 12
- net +3V0: track 17.4 -> 372.8 mm, vias 2 -> 11
- net VBUS: track 20.2 -> 325.8 mm, vias 2 -> 3
- net +10V: track 1.90 -> 251.8 mm, vias 0 -> 7
- net +3.3VA: track 5.41 -> 220.8 mm, vias 1 -> 6
- net -5V: track 70.8 -> 211.8 mm, vias 4 -> 8
- net Net-(SW402-B): track 0.00 -> 95.8 mm, vias 0 -> 2
- net D4_A: track 0.00 -> 89.6 mm, vias 0 -> 2
- net D3_A: track 0.00 -> 84.3 mm, vias 0 -> 2
- net Net-(SW403-B): track 0.00 -> 82.1 mm, vias 0 -> 1
- net D2_A: track 0.00 -> 79.9 mm, vias 0 -> 2
- net D7_A: track 0.00 -> 67.3 mm
- net D1_A: track 0.00 -> 65.8 mm, vias 0 -> 2
- net D8_A: track 0.00 -> 64.9 mm, vias 0 -> 2
- net D10_A: track 0.00 -> 64.1 mm, vias 0 -> 2
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- removed copper zone on In3.Cu, net GND
