File: VNA_Project/VNA_Project.kicad_pcb (KiCad board)
At the start: 6 copper layers, 200 x 200 mm, 231 parts, among them J201 USB_C_Receptacle_USB2.0_16P, J202 Jack-DC, J203 Screw_Terminal_01x01, J301 2x5 1.27mm, J302 Screw_Terminal_01x02, J401 Conn_Coaxial, J402 Conn_Coaxial, J403 Conn_Coaxial, J501 RJ45_Amphenol_RJMG1BD3B8K1ANR, SW201 SW_SPDT, SW202 SW_SPDT, SW301 SW_SPDT, SW401 SW_SPDT, SW402 SW_SPDT, SW403 SW_SPDT, U201 AP63205WU, U202 AP63203WU, U203 USBLC6-2SC6, U204 HT7533-1, U205 MIC5501-3.0YM5, U206 TPS54620RGYR, U207 MCP1804x-A002xOT, U301 TMP75AID, U302 TMP75AID, U303 STM32H730VBTx, U304 TMP75AID, U305 TL972IPWR, U401 LT1813CS8-TRPBF, U402 LT1813CS8-TRPBF, U403 AD9238BSTZ-20, U404 AD8138ARZ, U405 AD8138ARZ, U501 LAN8742A, U502 USBLC6-4SC6, Y301 STDCZS1-25M, Y501 STDCZS1-25M

Commit message: clearance changed
clearance changed
Routing:
- net Net-(C414-Pad1): track 39.8 -> 39.1 mm

Commit message: DRC silkscreen
fixed DRC and silkscreen
Parts:
- added G***: LOGO, LOGO, B.Cu at (357.7, 256.5)
- added G***: LOGO, LOGO, B.Cu at (367.9, 157.7)
- added G***: LOGO, LOGO, B.Cu at (358.0, 130.8)
- D301, D302, D303, D304, D305: footprint Diode_SMD:Infineon_SG-WLL-2-3_0.58x0.28_P0.36mm -> Diode_SMD:Nexperia_DSN0603-2_0.6x0.3mm_P0.4mm
- G***: moved to F.Cu
- moved G*** 2.98 mm to (367.9, 260.2), turned to 0 degrees
- moved D301 0.79 mm to (243.8, 296.5)
- moved SW301 0.69 mm to (273.0, 295.3)
- moved D305 0.14 mm to (257.6, 291.2)
Routing:
- net NRST: track 127.6 -> 131.6 mm
- net /Power/CC_2_pulldown: track 7.68 -> 10.6 mm
- net VBUS: track 325.8 -> 328.4 mm
- net /Power/CC_1_pulldown: track 7.66 -> 10.3 mm
- net /Ethernet/CRD: track 135.6 -> 137.6 mm
- net GND: track 259.7 -> 261.0 mm, vias 162 -> 161
- net +3.3V: track 99.8 -> 99.1 mm
- net Net-(SW301-B): track 4.85 -> 4.24 mm
Other:
- board text added: "+15V IN"
- board text added: "ETHERNET"
- board text added: "Flatrim Dreshaj NOV 2025"
- board text added: "HUBRIS VNA V1"
- board text added: "SWD"
- board text added: "https://github.com/fdreshaj/VNA_Design"
- board text removed: "-5V not included"
- board text removed: "15V IN"

Commit message: GRB BOM
GRB BOM
Parts:
- C203, C204, C207, C221, C222: footprint Capacitor_SMD:C_0805_2012Metric -> Capacitor_SMD:C_0603_1608Metric
Connections:
- net /Ethernet/CRD renamed /Ethernet [5]/CRD
- net /Ethernet/xtal2_eth renamed /Ethernet [5]/xtal2_eth
- net /MCU/CONN_NRST renamed /MCU [3]/CONN_NRST
- net /MCU/CONN_SWCLK renamed /MCU [3]/CONN_SWCLK
- net /MCU/CONN_SWDIO renamed /MCU [3]/CONN_SWDIO
- net /MCU/CONN_SWO renamed /MCU [3]/CONN_SWO
- net /MCU/analog decoupling renamed /MCU [3]/analog decoupling
- net /MCU/vref+ renamed /MCU [3]/vref+
- net /Power/5_volt_filt renamed /Power [2]/5_volt_filt
- net /Power/CC_1_pulldown renamed /Power [2]/CC_1_pulldown
- net /Power/CC_2_pulldown renamed /Power [2]/CC_2_pulldown
- net /Power/SW_POWER renamed /Power [2]/SW_POWER
- net /Power/usbc_d+ renamed /Power [2]/usbc_d+
- net /Power/usbc_d- renamed /Power [2]/usbc_d-
