File: VNA_Project/Power.kicad_sch (KiCad schematic)
At the start: 40 parts, among them J1 Jack-DC, J201 USB_C_Receptacle_USB2.0_16P, SW1 SW_SPDT, U10 MCP1804x-A002xOT, U11 AP7375-50SA-7, U202 USBLC6-2SC6, U204 HT7533-1, U6 MIC5501-3.0YM5, U9 AP63203WU

Commit message: VNA V1
FRONT END  FIRST PROTOTYPE SCHEMATIC DONE
Parts:
- removed C203: 1u, symbol Device:C
- removed C205: 10u, symbol Device:C
- removed D201: Green, symbol Device:LED
- removed R203: 1k, symbol Device:R
- removed U11: AP7375-50SA-7, SOT23_DIO_DOD, symbol Non_KiCad_Symbols:AP7375-50SA-7
- added C12, C13, C14: 68u, symbol Device:C
- added C15: 15u, symbol Device:C
- added C16, C24: 0.1u, symbol Device:C
- added C17: DNF, symbol Device:C
- added C19, C20, C21: 47u, symbol Device:C
- added C22: 0.01u, symbol Device:C
- added C23: 0.22u, symbol Device:C
- added C53: 100n, symbol Device:C
- added C54: 100p, symbol Device:C
- added C55, C56: 22u, symbol Device:C
- added C57: 10u, symbol Device:C
- added D11: Green, symbol Device:LED
- added J5: Screw_Terminal_01x01, symbol Connector:Screw_Terminal_01x01
- added L3, L4: 10u, symbol Device:L
- added R17: 162k, symbol Device:R
- added R18: 49.9, symbol Device:R
- added R19: 52.3k, symbol Device:R
- added R20: 10k, symbol Device:R
- added R21: 1.54k, symbol Device:R
- added R22: 158k, symbol Device:R
- added R23: 30.1k, symbol Device:R
- added R24: 1k, symbol Device:R
- added SW6: SW_SPDT, symbol Switch:SW_SPDT
- added TP4, TP5, TP6, TP7, TP8, TP9: TestPoint, symbol Connector:TestPoint
- added U15: TPS54620RGYR, TPS54620RGYR:QFN50P350X350X100-15N, symbol Non_KiCad_Symbols:TPS54620RGYR
- added U16: AP63205WU, Package_TO_SOT_SMD:TSOT-23-6, symbol Regulator_Switching:AP63205WU
Connections:
- net +15V: now also C57.1, U16.2 (EN), U16.3 (IN)
- net +5V: now also SW1.3 (C), C54.1, C55.1, C56.1, D11.2 (A), L4.2, R22.1; no longer SW1.1 (A)
- net GND: now also C12.2, C13.2, C14.2, C19.1, C20.1, C21.1, C55.2, C56.2, C57.2, L3.2, R18.1, R23.2, R24.2, TP7.1, TP9.1, U16.4 (GND)
- net VBUS: now also SW1.1 (A); no longer SW1.3 (C)
- net at C207.1, C25.1, C34.1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: now also C12.1, C13.1, C14.1, C15.1, C24.1, TP4.1, U15.4 (PVIN_4), U15.5 (PVIN_5), U15.6 (VIN)
- new net: C16.2, U15.13 (BOOT)
- new net: C53.1, L4.1, U16.5 (SW)
- new net: SW6.1 (A), TP5.1
- new net: C53.2, U16.6 (BST)
- new net: D11.1 (K), R24.1
- new net: C23.1, R21.1
- new net: R17.1, U15.1 (RT/CLK)
- new net: C22.1, U15.9 (SS/TR)
- new net: C17.1, R18.2, R19.1
- new net: C54.2, R22.2, R23.1, U16.1 (FB)
- new net: J5.1 (Pin_1), SW6.3 (C)
- new net -5V: C15.2, C19.2, C20.2, C21.2, C22.2, C23.2, C24.2, R17.2, R20.2, TP8.1, U15.15 (EXP), U15.2 (GND_2), U15.3 (GND_3)
- new net EN_inverting: SW6.2 (B), U15.10 (EN)
- new net boot_inv: C16.1, L3.1, TP6.1, U15.11 (PH_11), U15.12 (PH_12)
- new net comp_inv: R21.2, U15.8 (COMP)
- new net vsns_inv: C17.2, R19.2, R20.1, U15.7 (VSENSE)
- no-connect marks 3 -> 4
Other:
- note added: "-5V"
- note added: "15-5V"
- note added: "3-3.3V"
- note added: "5V"
- note added: "gnd"
- note removed: "AP7375-50SA-7"
- note removed: "Use X7R Caps"
- note removed: "Will be adding shielding and ESD straps on the board later on"
- moved on the sheet: C207, C208, C209, C211, C25, C26, C34, C35, C36, C37, C38, C39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

Commit message: footprints + initial layout shape
footprints + initial layout shape
Parts:
- C201: renamed from C57; footprint (none) -> Capacitor_SMD:C_0805_2012Metric
- C202: renamed from C34; footprint Capacitor_SMD:C_1206_3216Metric_Pad1.33x1.80mm_HandSolder -> Capacitor_SMD:C_0805_2012Metric
- C203: renamed from C204; footprint Capacitor_SMD:C_0402_1005Metric_Pad0.74x0.62mm_HandSolder -> Capacitor_SMD:C_0805_2012Metric
- C204: renamed from C53; footprint (none) -> Capacitor_SMD:C_0805_2012Metric
- C205: renamed from C207; footprint Capacitor_SMD:C_0603_1608Metric -> Capacitor_SMD:C_0805_2012Metric
- C206: renamed from C54; footprint (none) -> Capacitor_SMD:C_0805_2012Metric
- C207: renamed from C35; footprint Capacitor_SMD:C_1206_3216Metric_Pad1.33x1.80mm_HandSolder -> Capacitor_SMD:C_0805_2012Metric
- C208: footprint Capacitor_SMD:C_0603_1608Metric -> Capacitor_SMD:C_0805_2012Metric
- C209: renamed from C36; footprint Capacitor_SMD:C_1206_3216Metric_Pad1.33x1.80mm_HandSolder -> Capacitor_SMD:C_0805_2012Metric
- C210: renamed from C55; footprint (none) -> Capacitor_SMD:C_0805_2012Metric
- C211: renamed from C25; footprint (none) -> Capacitor_SMD:C_0805_2012Metric
- C213: renamed from C37; footprint Capacitor_SMD:C_1206_3216Metric_Pad1.33x1.80mm_HandSolder -> Capacitor_SMD:C_0805_2012Metric
- C214: renamed from C56; footprint (none) -> Capacitor_SMD:C_0805_2012Metric
- C216: renamed from C12; footprint (none) -> Capacitor_SMD:C_0805_2012Metric
- C217: renamed from C26; footprint (none) -> Capacitor_SMD:C_0805_2012Metric
- C218: renamed from C13; footprint (none) -> Capacitor_SMD:C_0805_2012Metric
- C219: renamed from C14; footprint (none) -> Capacitor_SMD:C_0805_2012Metric
- C220: renamed from C15; footprint (none) -> Capacitor_SMD:C_0805_2012Metric
- C221: renamed from C24; footprint (none) -> Capacitor_SMD:C_0805_2012Metric
- C222: renamed from C16; footprint (none) -> Capacitor_SMD:C_0805_2012Metric
- C223: renamed from C38; footprint (none) -> Capacitor_SMD:C_0805_2012Metric
- C224: renamed from C23; footprint (none) -> Capacitor_SMD:C_0805_2012Metric
- C225: renamed from C22; footprint (none) -> Capacitor_SMD:C_0805_2012Metric
- C226: renamed from C17; footprint (none) -> Capacitor_SMD:C_0805_2012Metric
- C227: renamed from C39; footprint (none) -> Capacitor_SMD:C_0805_2012Metric
- C228: renamed from C19; footprint (none) -> Capacitor_SMD:C_0805_2012Metric
- C229: renamed from C20; footprint (none) -> Capacitor_SMD:C_0805_2012Metric
- C230: renamed from C21; footprint (none) -> Capacitor_SMD:C_0805_2012Metric
- D201: renamed from D204; footprint (none) -> LED_SMD:LED_0603_1608Metric_Pad1.05x0.95mm_HandSolder
- D202: renamed from D4; footprint (none) -> LED_SMD:LED_0603_1608Metric_Pad1.05x0.95mm_HandSolder
- D203: renamed from D11; footprint (none) -> LED_SMD:LED_0603_1608Metric_Pad1.05x0.95mm_HandSolder
- D204: renamed from D202; footprint (none) -> LED_SMD:LED_0603_1608Metric_Pad1.05x0.95mm_HandSolder
- D205: renamed from D1; footprint (none) -> LED_SMD:LED_0603_1608Metric_Pad1.05x0.95mm_HandSolder
- D206: renamed from D5; footprint (none) -> LED_SMD:LED_0603_1608Metric_Pad1.05x0.95mm_HandSolder
- J202: renamed from J1; footprint (none) -> Connector_BarrelJack:BarrelJack_GCT_DCJ200-10-A_Horizontal
- J203: renamed from J5; footprint (none) -> TerminalBlock:TerminalBlock_MaiXu_MX126-5.0-02P_1x02_P5.00mm
- L201: renamed from L4; footprint (none) -> Inductor_SMD:L_0805_2012Metric_Pad1.15x1.40mm_HandSolder
- L202: footprint Inductor_SMD:L_0402_1005Metric -> Inductor_SMD:L_0805_2012Metric_Pad1.15x1.40mm_HandSolder
- L203: renamed from L2; footprint Inductor_SMD:L_Bourns_SDR0604 -> Inductor_SMD:L_0805_2012Metric_Pad1.15x1.40mm_HandSolder
- L204: renamed from L3; footprint (none) -> Inductor_SMD:L_0805_2012Metric_Pad1.15x1.40mm_HandSolder
- R201, R202: footprint Resistor_SMD:R_0402_1005Metric_Pad0.72x0.64mm_HandSolder -> Resistor_SMD:R_0603_1608Metric_Pad0.98x0.95mm_HandSolder
- R203: renamed from R208; footprint (none) -> Resistor_SMD:R_0603_1608Metric_Pad0.98x0.95mm_HandSolder
- R204: renamed from R22; footprint (none) -> Resistor_SMD:R_0603_1608Metric_Pad0.98x0.95mm_HandSolder
- R205: renamed from R23; footprint (none) -> Resistor_SMD:R_0603_1608Metric_Pad0.98x0.95mm_HandSolder
- R206: renamed from R38; footprint Resistor_SMD:R_0402_1005Metric_Pad0.72x0.64mm_HandSolder -> Resistor_SMD:R_0603_1608Metric_Pad0.98x0.95mm_HandSolder
- R207: renamed from R24; footprint (none) -> Resistor_SMD:R_0603_1608Metric_Pad0.98x0.95mm_HandSolder
- R208: renamed from R206; footprint (none) -> Resistor_SMD:R_0603_1608Metric_Pad0.98x0.95mm_HandSolder
- R209: renamed from R29; footprint (none) -> Resistor_SMD:R_0603_1608Metric_Pad0.98x0.95mm_HandSolder
- R210: renamed from R17; footprint (none) -> Resistor_SMD:R_0603_1608Metric_Pad0.98x0.95mm_HandSolder
- R211: renamed from R21; footprint (none) -> Resistor_SMD:R_0603_1608Metric_Pad0.98x0.95mm_HandSolder
- R212: renamed from R18; footprint (none) -> Resistor_SMD:R_0603_1608Metric_Pad0.98x0.95mm_HandSolder
- R213: renamed from R19; footprint (none) -> Resistor_SMD:R_0603_1608Metric_Pad0.98x0.95mm_HandSolder
- R214: renamed from R20; footprint (none) -> Resistor_SMD:R_0603_1608Metric_Pad0.98x0.95mm_HandSolder
- R215: renamed from R39; footprint (none) -> Resistor_SMD:R_0603_1608Metric_Pad0.98x0.95mm_HandSolder
- SW202: renamed from SW6; footprint (none) -> Button_Switch_THT:SW_Slide_SPDT_Straight_CK_OS102011MS2Q
- TP201: renamed from TP4; footprint (none) -> TestPoint:TestPoint_Pad_D4.0mm
- TP202: renamed from TP9; footprint (none) -> TestPoint:TestPoint_Pad_D4.0mm
- TP203: renamed from TP6; footprint (none) -> TestPoint:TestPoint_Pad_D4.0mm
- TP204: renamed from TP5; footprint (none) -> TestPoint:TestPoint_Pad_D4.0mm
- TP205: renamed from TP7; footprint (none) -> TestPoint:TestPoint_Pad_D4.0mm
- TP206: renamed from TP8; footprint (none) -> TestPoint:TestPoint_Pad_D4.0mm
- U201: renamed from U16; footprint Package_TO_SOT_SMD:TSOT-23-6 -> Package_TO_SOT_SMD:TSOT-23-6_HandSoldering
- U202: renamed from U9; footprint Package_TO_SOT_SMD:TSOT-23-6 -> Package_TO_SOT_SMD:TSOT-23-6_HandSoldering
- U203: renamed from U202; footprint Package_TO_SOT_SMD:SOT-23-6 -> Package_TO_SOT_SMD:SOT-23-6_Handsoldering
- U204: footprint Package_TO_SOT_SMD:SOT-89-3 -> Package_TO_SOT_SMD:SOT-89-3_Handsoldering
- U205: renamed from U6; footprint Package_TO_SOT_SMD:SOT-23-5 -> Package_TO_SOT_SMD:SOT-23-5_HandSoldering
- U206: renamed from U15; footprint TPS54620RGYR:QFN50P350X350X100-15N -> NonKiCad_footprints:TPS54620RGYR
- U207: renamed from U10; footprint Package_TO_SOT_SMD:SOT-23-5 -> Package_TO_SOT_SMD:SOT-23-5_HandSoldering
- renumbered C209 to C212, C211 to C215, SW1 to SW201
Other:
- moved on the sheet: C201

Commit message: layout
layout
Parts:
- L201, L202, L203, L204: footprint Inductor_SMD:L_0805_2012Metric_Pad1.15x1.40mm_HandSolder -> Inductor_SMD:L_APV_ANR6020
Connections:
- net SW_POWER: now reaches C202.1, C205.1, C211.1, C216.1, C218.1, C219.1, C220.1, C221.1, L202.1, SW201.2 (B), TP201.1, U202.2 (EN), U202.3 (IN), U205.1 (VIN), U205.3 (EN), U206.4 (PVIN_4), U206.5 (PVIN_5), U206.6 (VIN)
Changed lines of the file:
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@@
 		)
 	)
+	(label "SW_POWER"
+		(at 58.42 257.81 0)
+		(effects
+			(font
+				(size 1.27 1.27)
+			)
+			(justify left bottom)
+		)
+	)
 	(label "CC_1_pulldown"
 		(at 59.69 116.84 0)
@@
 			)
 		)
-		(property "Footprint" "Inductor_SMD:L_0805_2012Metric_Pad1.15x1.40mm_HandSolder"
+		(property "Footprint" "Inductor_SMD:L_APV_ANR6020"
 			(at 102.87 218.44 0)
 			(effects
@@
 			)
 		)
-		(property "Footprint" "Inductor_SMD:L_0805_2012Metric_Pad1.15x1.40mm_HandSolder"
+		(property "Footprint" "Inductor_SMD:L_APV_ANR6020"
 			(at 93.98 27.94 0)
 			(effects
@@
 			)
 		)
-		(property "Footprint" "Inductor_SMD:L_0805_2012Metric_Pad1.15x1.40mm_HandSolder"
+		(property "Footprint" "Inductor_SMD:L_APV_ANR6020"
 			(at 313.69 100.33 0)
 			(effects
@@
 			)
 		)
-		(property "Footprint" "Inductor_SMD:L_0805_2012Metric_Pad1.15x1.40mm_HandSolder"
+		(property "Footprint" "Inductor_SMD:L_APV_ANR6020"
 			(at 110.49 255.27 0)
 			(effects

Commit message: GRB BOM
GRB BOM
Parts:
- C203, C204, C207, C221, C222: footprint Capacitor_SMD:C_0805_2012Metric -> Capacitor_SMD:C_0603_1608Metric
Changed lines of the file:
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@@
 			)
 		)
-		(property "Footprint" "Capacitor_SMD:C_0805_2012Metric"
+		(property "Footprint" "Capacitor_SMD:C_0603_1608Metric"
 			(at 202.8952 116.84 0)
 			(effects
@@
 			)
 		)
-		(property "Footprint" "Capacitor_SMD:C_0805_2012Metric"
+		(property "Footprint" "Capacitor_SMD:C_0603_1608Metric"
 			(at 245.11 106.9848 0)
 			(effects
@@
 			)
 		)
-		(property "Footprint" "Capacitor_SMD:C_0805_2012Metric"
+		(property "Footprint" "Capacitor_SMD:C_0603_1608Metric"
 			(at 82.2452 35.56 0)
 			(effects
@@
 			)
 		)
-		(property "Footprint" "Capacitor_SMD:C_0805_2012Metric"
+		(property "Footprint" "Capacitor_SMD:C_0603_1608Metric"
 			(at 71.12 99.3648 0)
 			(effects
@@
 			)
 		)
-		(property "Footprint" "Capacitor_SMD:C_0805_2012Metric"
+		(property "Footprint" "Capacitor_SMD:C_0603_1608Metric"
 			(at 102.87 257.81 0)
 			(effects
