File: VNA_Project/VCO_Design/VCO_Design.kicad_sch (KiCad schematic)
At the start: 25 parts, among them J101 Screw_Terminal_01x02, J102 Screw_Terminal_01x02, Q101 NPN

Commit message: vco design
vco design
Parts:
- removed Q101: NPN, symbol Simulation_SPICE:NPN
- removed R105: 50, symbol Device:R
- added J103: Conn_Coaxial, Connector_Coaxial:SMA_Amphenol_901-144_Vertical, symbol Connector:Conn_Coaxial
- added Q101: BFP620, NonKiCad_footprints:bfptransistor, symbol Transistor_BJT:BC240
- C101, C102, C103, C104, C105, C106, C107, C108, C109, C110: footprint (none) -> Capacitor_SMD:C_0603_1608Metric_Pad1.08x0.95mm_HandSolder
- D101, D102: footprint (none) -> NonKiCad_footprints:SMV1247
- J101, J102: footprint (none) -> TerminalBlock:TerminalBlock_Altech_AK300-2_P5.00mm
- L103, L104, L105, L106, L107: footprint (none) -> Inductor_SMD:L_0603_1608Metric_Pad1.05x0.95mm_HandSolder
- R101, R102, R103, R104: footprint (none) -> Resistor_SMD:R_0603_1608Metric_Pad0.98x0.95mm_HandSolder
Connections:
- net GND: now also J103.2 (Ext)
- net at C101.1, R101.2, R103.1: now also Q101.3 (B)
- net at C105.1, R104.1: now also Q101.2 (E)
- net at C104.1, R102.2: now also Q101.1 (C)
- net at C104.2, C106.2, L103.2: now also J103.1 (In)
